File: eagle/main.sch (EAGLE design)
At the start: 33 parts, among them IC1 TS5205, Q1 SI4840DY, Q5 SI4840DY, U1 SN74AHC1G00DCKR, U2 SN74AHC1G00DCKR, U3 SN74AHC1G00DCKR

Commit message: update
Parts:
- removed T1, T2: (no value), transistor:-NPN-TO92
- added T3, T4: (no value), transistor:BC817-40-NPN-SOT23-BEC
- R1, R2, R3, R4, R6, R8: device resistor:R-US_0204/2V -> resistor:R-US_M0805
- R5, R7: value 400K -> 390K; device resistor:R-US_0204/2V -> resistor:R-US_M0805
Connections:
- net GND: now also T3.E, T4.E; no longer T1.E, T2.E
- net N$1: now also T3.C; no longer T1.C
- net N$2: now also T4.C; no longer T2.C
- net N$3: now also T4.B; no longer T2.B
- net N$6: now also T3.B; no longer T1.B
Other:
- note added: "voltage monitoring paths 4.9:1 divider"
- note removed: "TODO: choose FET"
- note removed: "TODO: choose resistors"
- note removed: "voltage monitoring paths"
Changed lines of the file:
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@@
 <part name="D2" library="diode" deviceset="1N4148" device="DO35-7"/>
 <part name="C1" library="rcl" deviceset="CPOL-US" device="085CS-1AR"/>
-<part name="R2" library="resistor" deviceset="R-US_" device="0204/2V" value="100K"/>
-<part name="T1" library="transistor" deviceset="*-NPN-" device="TO92"/>
-<part name="R4" library="resistor" deviceset="R-US_" device="0204/2V" value="10K"/>
+<part name="R2" library="resistor" deviceset="R-US_" device="M0805" value="100K"/>
+<part name="R4" library="resistor" deviceset="R-US_" device="M0805" value="10K"/>
 <part name="U1" library="TI-SN74AHC1G00DCKR@E" deviceset="SN74AHC1G00DCKR" device=""/>
 <part name="U2" library="TI-SN74AHC1G00DCKR@E" deviceset="SN74AHC1G00DCKR" device=""/>
@@
 <part name="D7" library="diode" deviceset="1N4148" device="DO35-7"/>
 <part name="SUPPLY1" library="supply2" deviceset="GND" device=""/>
-<part name="R1" library="resistor" deviceset="R-US_" device="0204/2V" value="100K"/>
-<part name="T2" library="transistor" deviceset="*-NPN-" device="TO92"/>
-<part name="R3" library="resistor" deviceset="R-US_" device="0204/2V" value="10K"/>
+<part name="R1" library="resistor" deviceset="R-US_" device="M0805" value="100K"/>
+<part name="R3" library="resistor" deviceset="R-US_" device="M0805" value="10K"/>
 <part name="SUPPLY2" library="supply2" deviceset="GND" device=""/>
 <part name="U$2" library="Teensy3.0" deviceset="TEENSY_3.0_ALLPINS" device=""/>
 <part name="D3" library="diode" deviceset="1N4148" device="DO35-7"/>
 <part name="SPI_CON" library="pinhead" deviceset="PINHD-1X6" device=""/>
-<part name="R5" library="resistor" deviceset="R-US_" device="0204/2V" value="400K"/>
-<part name="R6" library="resistor" deviceset="R-US_" device="0204/2V" value="100K"/>
+<part name="R5" library="resistor" deviceset="R-US_" device="M0805" value="390K"/>
+<part name="R6" library="resistor" deviceset="R-US_" device="M0805" value="100K"/>
 <part name="SUPPLY3" library="supply2" deviceset="GND" device=""/>
-<part name="R7" library="resistor" deviceset="R-US_" device="0204/2V" value="400K"/>
-<part name="R8" library="resistor" deviceset="R-US_" device="0204/2V" value="100K"/>
+<part name="R7" library="resistor" deviceset="R-US_" device="M0805" value="390K"/>
+<part name="R8" library="resistor" deviceset="R-US_" device="M0805" value="100K"/>
 <part name="SUPPLY4" library="supply2" deviceset="GND" device=""/>
 <part name="IC1" library="v-reg" deviceset="TS5205" device=""/>
@@
 <part name="Q5" library="transistor-fet" deviceset="SI4840DY" device=""/>
 <part name="Q1" library="transistor-fet" deviceset="SI4840DY" device=""/>
+<part name="T3" library="transistor" deviceset="*-NPN-" device="SOT23-BEC" technology="BC817-40"/>
+<part name="T4" library="transistor" deviceset="*-NPN-" device="SOT23-BEC" technology="BC817-40"/>
 </parts>
 <sheets>
@@
 freq:</text>
 <text x="254" y="7.62" size="1.778" layer="97">TODO: choose Schottky diodes</text>
-<text x="320.04" y="15.24" size="1.778" layer="97">power paths</text>
+<text x="320.04" y="2.54" size="1.778" layer="97">power paths</text>
 <text x="137.16" y="7.62" size="1.778" layer="97">TODO: choose diodes</text>
-<text x="391.16" y="7.62" size="1.778" layer="97">voltage monitoring paths</text>
+<text x="391.16" y="2.54" size="1.778" layer="97">voltage monitoring paths
+4.9:1 divider</text>
 <text x="226.06" y="10.16" size="1.778" layer="97">TODO: choose caps</text>
 <text x="254" y="5.08" size="1.778" layer="97">TODO: choose caps</text>
 <text x="40.64" y="-45.72" size="1.778" layer="97">SPI connector</text>
-<text x="320.04" y="7.62" size="1.778" layer="97">TODO: choose FET</text>
-<text x="320.04" y="5.08" size="1.778" layer="97">TODO: choose resistors</text>
-<text x="391.16" y="2.54" size="1.778" layer="97">TODO: choose resistors</text>
 <text x="40.64" y="10.16" size="1.778" layer="97">TODO: choose connectors</text>
 <text x="365.76" y="-20.32" size="1.778" layer="97">SI4166DY</text>
@@
 <instance part="C1" gate="G$1" x="162.56" y="-10.16"/>
 <instance part="R2" gate="G$1" x="340.36" y="-27.94"/>
-<instance part="T1" gate="G$1" x="350.52" y="-27.94" smashed="yes">
-<attribute name="NAME" x="345.44" y="-25.4" size="1.778" layer="95"/>
-<attribute name="VALUE" x="340.36" y="-22.86" size="1.778" layer="96"/>
-</instance>
 <instance part="R4" gate="G$1" x="353.06" y="-12.7" rot="R270"/>
 <instance part="U1" gate="A" x="93.98" y="-10.16"/>
@@
 <instance part="SUPPLY1" gate="GND" x="353.06" y="-38.1"/>
 <instance part="R1" gate="G$1" x="340.36" y="-71.12"/>
-<instance part="T2" gate="G$1" x="350.52" y="-71.12" smashed="yes">
-<attribute name="NAME" x="345.44" y="-68.58" size="1.778" layer="95"/>
-<attribute name="VALUE" x="340.36" y="-66.04" size="1.778" layer="96"/>
-</instance>
 <instance part="R3" gate="G$1" x="353.06" y="-55.88" rot="R270"/>
 <instance part="SUPPLY2" gate="GND" x="353.06" y="-81.28"/>
@@
 <attribute name="NAME" x="365.76" y="-60.96" size="1.778" layer="95"/>
 </instance>
+<instance part="T3" gate="G$1" x="350.52" y="-27.94"/>
+<instance part="T4" gate="G$1" x="350.52" y="-71.12"/>
 </instances>
 <busses>
@@
 </segment>
 <segment>
-<pinref part="T1" gate="G$1" pin="E"/>
 <wire x1="353.06" y1="-33.02" x2="353.06" y2="-35.56" width="0.1524" layer="91"/>
 <pinref part="SUPPLY1" gate="GND" pin="GND"/>
-</segment>
-<segment>
-<pinref part="T2" gate="G$1" pin="E"/>
+<pinref part="T3" gate="G$1" pin="E"/>
+</segment>
+<segment>
 <wire x1="353.06" y1="-76.2" x2="353.06" y2="-78.74" width="0.1524" layer="91"/>
 <pinref part="SUPPLY2" gate="GND" pin="GND"/>
+<pinref part="T4" gate="G$1" pin="E"/>
 </segment>
 <segment>
@@
 <segment>
 <pinref part="R4" gate="G$1" pin="2"/>
-<pinref part="T1" gate="G$1" pin="C"/>
 <wire x1="353.06" y1="-17.78" x2="353.06" y2="-20.32" width="0.1524" layer="91"/>
 <wire x1="353.06" y1="-20.32" x2="353.06" y2="-22.86" width="0.1524" layer="91"/>
@@
 <junction x="353.06" y="-20.32"/>
 <pinref part="Q5" gate="G$1" pin="G"/>
+<pinref part="T3" gate="G$1" pin="C"/>
 </segment>
 </net>
@@
 <segment>
 <pinref part="R2" gate="G$1" pin="2"/>
-<pinref part="T1" gate="G$1" pin="B"/>
 <wire x1="345.44" y1="-27.94" x2="347.98" y2="-27.94" width="0.1524" layer="91"/>
+<pinref part="T3" gate="G$1" pin="B"/>
 </segment>
 </net>
@@
 <segment>
 <pinref part="R3" gate="G$1" pin="2"/>
-<pinref part="T2" gate="G$1" pin="C"/>
 <wire x1="353.06" y1="-60.96" x2="353.06" y2="-63.5" width="0.1524" layer="91"/>
 <wire x1="353.06" y1="-63.5" x2="353.06" y2="-66.04" width="0.1524" layer="91"/>
@@
 <junction x="353.06" y="-63.5"/>
 <pinref part="Q1" gate="G$1" pin="G"/>
+<pinref part="T4" gate="G$1" pin="C"/>
 </segment>
 </net>
@@
 <segment>
 <pinref part="R1" gate="G$1" pin="2"/>
-<pinref part="T2" gate="G$1" pin="B"/>
 <wire x1="345.44" y1="-71.12" x2="347.98" y2="-71.12" width="0.1524" layer="91"/>
-</segment>
-</net>
+<pinref part="T4" gate="G$1" pin="B"/>
+</segment>
+</net>

Commit message: update
Parts:
- removed C4: (no value), rcl:CPOL-US085CS-1AR
- added C7: 10u, rcl:CPOL-US085CS-1AR
- added C8: 100UF, Panasonic-EEEFK_EEEFP:EEE-FK1E101XP-CASE-D8
- C1: value (none) -> 2.2u
- C5, C6: value (none) -> 10u
Connections:
- net GND: now also C7.-, C8.2; no longer C4.-
- net LOAD_V+: now also C8.1; no longer C4.+
- net PUMP_V+: now also C7.+
Changed lines of the file:
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@@
 <part name="D1" library="diode" deviceset="1N4148" device="DO35-7"/>
 <part name="D2" library="diode" deviceset="1N4148" device="DO35-7"/>
-<part name="C1" library="rcl" deviceset="CPOL-US" device="085CS-1AR"/>
+<part name="C1" library="rcl" deviceset="CPOL-US" device="085CS-1AR" value="2.2u"/>
 <part name="R2" library="resistor" deviceset="R-US_" device="M0805" value="100K"/>
 <part name="R4" library="resistor" deviceset="R-US_" device="M0805" value="10K"/>
@@
 <part name="U3" library="TI-SN74AHC1G00DCKR@E" deviceset="SN74AHC1G00DCKR" device=""/>
 <part name="C3" library="rcl" deviceset="CPOL-US" device="085CS-1AR" value="2.2u"/>
-<part name="C4" library="rcl" deviceset="CPOL-US" device="085CS-1AR"/>
 <part name="D4" library="diode" deviceset="1N4148" device="DO35-7"/>
 <part name="D6" library="diode" deviceset="1N4148" device="DO35-7"/>
-<part name="C5" library="rcl" deviceset="CPOL-US" device="085CS-1AR"/>
-<part name="C6" library="rcl" deviceset="CPOL-US" device="085CS-1AR"/>
+<part name="C5" library="rcl" deviceset="CPOL-US" device="085CS-1AR" value="10u"/>
+<part name="C6" library="rcl" deviceset="CPOL-US" device="085CS-1AR" value="10u"/>
 <part name="D7" library="diode" deviceset="1N4148" device="DO35-7"/>
 <part name="SUPPLY1" library="supply2" deviceset="GND" device=""/>
@@
 <part name="T3" library="transistor" deviceset="*-NPN-" device="SOT23-BEC" technology="BC817-40"/>
 <part name="T4" library="transistor" deviceset="*-NPN-" device="SOT23-BEC" technology="BC817-40"/>
+<part name="C7" library="rcl" deviceset="CPOL-US" device="085CS-1AR" value="10u"/>
+<part name="C8" library="Panasonic-EEEFK_EEEFP" deviceset="EEE-" device="-CASE-D8" technology="FK1E101XP" value="100UF"/>
 </parts>
 <sheets>
@@
 output: 4V, 150mA</text>
 <text x="137.16" y="10.16" size="1.778" layer="97">TODO: choose caps</text>
-<text x="226.06" y="15.24" size="1.778" layer="97">load tank cap</text>
+<text x="226.06" y="10.16" size="1.778" layer="97">load tank cap</text>
 <text x="254" y="12.7" size="1.778" layer="97">Dickson charge pump
 output: input + 5V
@@
 <text x="391.16" y="2.54" size="1.778" layer="97">voltage monitoring paths
 4.9:1 divider</text>
-<text x="226.06" y="10.16" size="1.778" layer="97">TODO: choose caps</text>
 <text x="254" y="5.08" size="1.778" layer="97">TODO: choose caps</text>
 <text x="40.64" y="-45.72" size="1.778" layer="97">SPI connector</text>
@@
 <instance part="U3" gate="A" x="93.98" y="-55.88"/>
 <instance part="C3" gate="G$1" x="203.2" y="-10.16"/>
-<instance part="C4" gate="G$1" x="241.3" y="0"/>
 <instance part="D4" gate="G$1" x="279.4" y="-2.54" smashed="yes">
 <attribute name="NAME" x="281.94" y="-2.0574" size="1.778" layer="95"/>
@@
 <instance part="T3" gate="G$1" x="350.52" y="-27.94"/>
 <instance part="T4" gate="G$1" x="350.52" y="-71.12"/>
+<instance part="C7" gate="G$1" x="294.64" y="-7.62"/>
+<instance part="C8" gate="A" x="241.3" y="2.54" smashed="yes" rot="R270">
+<attribute name="NAME" x="244.0686" y="0.9144" size="2.0828" layer="95" ratio="10" rot="SR0"/>
+<attribute name="VALUE" x="241.935" y="-5.6896" size="2.0828" layer="96" ratio="10" rot="SR0"/>
+</instance>
 </instances>
 <busses>
@@
 </segment>
 <segment>
-<pinref part="C4" gate="G$1" pin="-"/>
 <wire x1="241.3" y1="-5.08" x2="241.3" y2="-7.62" width="0.1524" layer="91"/>
 <wire x1="241.3" y1="-7.62" x2="226.06" y2="-7.62" width="0.1524" layer="91"/>
 <label x="226.06" y="-7.62" size="1.778" layer="95"/>
+<pinref part="C8" gate="A" pin="2"/>
 </segment>
 <segment>
@@
 <pinref part="SUPPLY4" gate="GND" pin="GND"/>
 <wire x1="408.94" y1="-73.66" x2="408.94" y2="-76.2" width="0.1524" layer="91"/>
+</segment>
+<segment>
+<pinref part="C7" gate="G$1" pin="-"/>
+<wire x1="294.64" y1="-12.7" x2="294.64" y2="-20.32" width="0.1524" layer="91"/>
+<wire x1="294.64" y1="-20.32" x2="254" y2="-20.32" width="0.1524" layer="91"/>
+<label x="254" y="-20.32" size="1.778" layer="95"/>
 </segment>
 </net>
@@
 </segment>
 <segment>
-<pinref part="C4" gate="G$1" pin="+"/>
 <wire x1="241.3" y1="2.54" x2="241.3" y2="5.08" width="0.1524" layer="91"/>
 <wire x1="241.3" y1="5.08" x2="226.06" y2="5.08" width="0.1524" layer="91"/>
 <label x="226.06" y="5.08" size="1.778" layer="95"/>
+<pinref part="C8" gate="A" pin="1"/>
 </segment>
 <segment>
@@
 <segment>
 <pinref part="D7" gate="G$1" pin="C"/>
-<wire x1="292.1" y1="-2.54" x2="307.34" y2="-2.54" width="0.1524" layer="91"/>
+<wire x1="292.1" y1="-2.54" x2="294.64" y2="-2.54" width="0.1524" layer="91"/>
 <label x="297.18" y="-2.54" size="1.778" layer="95"/>
-</segment>
-<segment>
+<pinref part="C7" gate="G$1" pin="+"/>
+<wire x1="294.64" y1="-2.54" x2="307.34" y2="-2.54" width="0.1524" layer="91"/>
+<wire x1="294.64" y1="-5.08" x2="294.64" y2="-2.54" width="0.1524" layer="91"/>
+<junction x="294.64" y="-2.54"/>
+</segment>
+<segment>
