File: eagle/main.sch (EAGLE design)
At the start: 34 parts, among them IC1 TS5205, Q1 SI4840DY, Q5 SI4840DY, U1 SN74AHC1G00DCKR, U2 SN74AHC1G00DCKR, U3 SN74AHC1G00DCKR

Commit message: update
Parts:
- C1, C3: device rcl:CPOL-US085CS-1AR -> rcl:C-USC1210K
- C2: device resistor:C-EU025-024X044 -> rcl:C-EUC0805K
Connections:
- net GND: now also C1.2, C3.2; no longer C1.-, C3.-
- net LOGIC_V+: now also C3.1; no longer C3.+
- net POW01_V+: now also C1.1; no longer C1.+
Changed lines of the file:
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@@
 <part name="D1" library="diode" deviceset="1N4148" device="DO35-7"/>
 <part name="D2" library="diode" deviceset="1N4148" device="DO35-7"/>
-<part name="C1" library="rcl" deviceset="CPOL-US" device="085CS-1AR" value="2.2u"/>
+<part name="C1" library="rcl" deviceset="C-US" device="C1210K" value="2.2u"/>
 <part name="R2" library="resistor" deviceset="R-US_" device="M0805" value="100K"/>
 <part name="R4" library="resistor" deviceset="R-US_" device="M0805" value="10K"/>
@@
 <part name="U2" library="TI-SN74AHC1G00DCKR@E" deviceset="SN74AHC1G00DCKR" device=""/>
 <part name="U3" library="TI-SN74AHC1G00DCKR@E" deviceset="SN74AHC1G00DCKR" device=""/>
-<part name="C3" library="rcl" deviceset="CPOL-US" device="085CS-1AR" value="2.2u"/>
+<part name="C3" library="rcl" deviceset="C-US" device="C1210K" value="2.2u"/>
 <part name="D4" library="diode" deviceset="1N4148" device="DO35-7"/>
 <part name="D6" library="diode" deviceset="1N4148" device="DO35-7"/>
@@
 <part name="SUPPLY4" library="supply2" deviceset="GND" device=""/>
 <part name="IC1" library="v-reg" deviceset="TS5205" device=""/>
-<part name="C2" library="resistor" deviceset="C-EU" device="025-024X044" value="470p"/>
+<part name="C2" library="rcl" deviceset="C-EU" device="C0805K" value="470p"/>
 <part name="Q5" library="transistor-fet" deviceset="SI4840DY" device=""/>
 <part name="Q1" library="transistor-fet" deviceset="SI4840DY" device=""/>
@@
 input: 5V to 16V
 output: 4V, 150mA</text>
-<text x="137.16" y="10.16" size="1.778" layer="97">TODO: choose caps</text>
 <text x="226.06" y="10.16" size="1.778" layer="97">load tank cap</text>
 <text x="254" y="12.7" size="1.778" layer="97">Dickson charge pump
@@
 <text x="254" y="7.62" size="1.778" layer="97">TODO: choose Schottky diodes</text>
 <text x="320.04" y="2.54" size="1.778" layer="97">power paths</text>
-<text x="137.16" y="7.62" size="1.778" layer="97">TODO: choose diodes</text>
+<text x="137.16" y="10.16" size="1.778" layer="97">TODO: choose diodes</text>
 <text x="391.16" y="2.54" size="1.778" layer="97">voltage monitoring paths
 4.9:1 divider</text>
@@
 </segment>
 <segment>
-<pinref part="C1" gate="G$1" pin="-"/>
+<pinref part="C1" gate="G$1" pin="2"/>
 <wire x1="162.56" y1="-15.24" x2="162.56" y2="-17.78" width="0.1524" layer="91"/>
 <wire x1="162.56" y1="-17.78" x2="137.16" y2="-17.78" width="0.1524" layer="91"/>
@@
 <wire x1="170.18" y1="-5.08" x2="170.18" y2="-17.78" width="0.1524" layer="91"/>
 <junction x="170.18" y="-17.78"/>
-<pinref part="C3" gate="G$1" pin="-"/>
+<pinref part="C3" gate="G$1" pin="2"/>
 <wire x1="203.2" y1="-15.24" x2="203.2" y2="-17.78" width="0.1524" layer="91"/>
 <pinref part="C2" gate="G$1" pin="2"/>
@@
 <wire x1="157.48" y1="-2.54" x2="162.56" y2="-2.54" width="0.1524" layer="91"/>
 <junction x="157.48" y="-2.54"/>
-<pinref part="C1" gate="G$1" pin="+"/>
+<pinref part="C1" gate="G$1" pin="1"/>
 <wire x1="162.56" y1="-2.54" x2="162.56" y2="-7.62" width="0.1524" layer="91"/>
 <wire x1="157.48" y1="-5.08" x2="157.48" y2="-10.16" width="0.1524" layer="91"/>
@@
 <wire x1="190.5" y1="5.08" x2="193.04" y2="5.08" width="0.1524" layer="91"/>
 <junction x="193.04" y="5.08"/>
-<pinref part="C3" gate="G$1" pin="+"/>
+<pinref part="C3" gate="G$1" pin="1"/>
 <wire x1="203.2" y1="5.08" x2="203.2" y2="-7.62" width="0.1524" layer="91"/>
 <junction x="203.2" y="5.08"/>

Commit message: update
Other:
- note added: "TODO: choose diodes (non Schottky)"
- note removed: "TODO: choose diodes"
Changed lines of the file:
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@@
 <text x="254" y="7.62" size="1.778" layer="97">TODO: choose Schottky diodes</text>
 <text x="320.04" y="2.54" size="1.778" layer="97">power paths</text>
-<text x="137.16" y="10.16" size="1.778" layer="97">TODO: choose diodes</text>
+<text x="137.16" y="10.16" size="1.778" layer="97">TODO: choose diodes (non Schottky)</text>
 <text x="391.16" y="2.54" size="1.778" layer="97">voltage monitoring paths
 4.9:1 divider</text>

Commit message: schottky diodes
Parts:
- removed D1, D2, D3: 1N4148DO35-7, diode:1N4148DO35-7
- added D5, D8, D9: (no value), diode:DIODE-DO214AC
- C1, C3: value 2.2u -> 4.7u
Connections:
- net LOGIC_V+: now also D9.A; no longer D3.A
- net POW01_V+: now also D5.C, D8.C; no longer D1.C, D2.C
- net POW0_V+: now also D5.A; no longer D1.A
- net POW1_V+: now also D8.A; no longer D2.A
- net SPI_V+: now also D9.C; no longer D3.C
Other:
- note added: "TS5205 LDK220"
- note added: "logic power supply, OR redundancy input: 5V to 16V output: 4V, 150mA (TS5205) output: 4V, 200mA (LDK220)"
- note removed: "logic power supply, OR redundancy input: 5V to 16V output: 4V, 150mA"

Commit message: update board
Parts:
- removed C7: 10u, rcl:CPOL-US085CS-1AR
- removed D4, D6, D7: 1N4148DO35-7, diode:1N4148DO35-7
- added C4: 4.7u, rcl:C-USC1210K
- added D1, D2, D3: (no value), diode:DIODE-DO214AC
- C5, C6: value 10u -> 4.7u; device rcl:CPOL-US085CS-1AR -> rcl:C-USC1210K
Connections:
- net GND: now also C6.2; no longer C7.-
- net N$4: now also C4.1, D1.C, D2.A; no longer C5.+, D4.A, D6.C
- net N$5: now also C5.1, D2.C, D3.A; no longer C6.+, D4.C, D7.A
- net POW01_V+: now also D1.A; no longer D6.A
- net PUMP_PWM: now also C4.2; no longer C5.-
- net PUMP_PWM#: now also C5.2; no longer C6.-
- net PUMP_V+: now also C6.1, D3.C; no longer C7.+, D7.C
Other:
- note removed: "TODO: choose Schottky diodes"
- note removed: "TODO: choose diodes (non Schottky)"
Changed lines of the file:
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@@
 <part name="U3" library="TI-SN74AHC1G00DCKR@E" deviceset="SN74AHC1G00DCKR" device=""/>
 <part name="C3" library="rcl" deviceset="C-US" device="C1210K" value="4.7u"/>
-<part name="D4" library="diode" deviceset="1N4148" device="DO35-7"/>
-<part name="D6" library="diode" deviceset="1N4148" device="DO35-7"/>
-<part name="C5" library="rcl" deviceset="CPOL-US" device="085CS-1AR" value="10u"/>
-<part name="C6" library="rcl" deviceset="CPOL-US" device="085CS-1AR" value="10u"/>
-<part name="D7" library="diode" deviceset="1N4148" device="DO35-7"/>
 <part name="SUPPLY1" library="supply2" deviceset="GND" device=""/>
 <part name="R1" library="resistor" deviceset="R-US_" device="M0805" value="100K"/>
@@
 <part name="T3" library="transistor" deviceset="*-NPN-" device="SOT23-BEC" technology="BC817-40"/>
 <part name="T4" library="transistor" deviceset="*-NPN-" device="SOT23-BEC" technology="BC817-40"/>
-<part name="C7" library="rcl" deviceset="CPOL-US" device="085CS-1AR" value="10u"/>
 <part name="C8" library="Panasonic-EEEFK_EEEFP" deviceset="EEE-" device="-CASE-D8" technology="FK1E101XP" value="100UF"/>
 <part name="D5" library="diode" deviceset="DIODE-" device="DO214AC"/>
 <part name="D8" library="diode" deviceset="DIODE-" device="DO214AC"/>
 <part name="D9" library="diode" deviceset="DIODE-" device="DO214AC"/>
+<part name="C4" library="rcl" deviceset="C-US" device="C1210K" value="4.7u"/>
+<part name="C5" library="rcl" deviceset="C-US" device="C1210K" value="4.7u"/>
+<part name="C6" library="rcl" deviceset="C-US" device="C1210K" value="4.7u"/>
+<part name="D1" library="diode" deviceset="DIODE-" device="DO214AC"/>
+<part name="D2" library="diode" deviceset="DIODE-" device="DO214AC"/>
+<part name="D3" library="diode" deviceset="DIODE-" device="DO214AC"/>
 </parts>
 <sheets>
@@
  1     1      0        1       1</text>
 <text x="40.64" y="15.24" size="1.778" layer="97">power supply connectors</text>
-<text x="137.16" y="15.24" size="1.778" layer="97">logic power supply, OR redundancy
+<text x="137.16" y="12.7" size="1.778" layer="97">logic power supply, OR redundancy
 input: 5V to 16V
 output: 4V, 150mA (TS5205)
 output: 4V, 200mA (LDK220)</text>
 <text x="226.06" y="10.16" size="1.778" layer="97">load tank cap</text>
-<text x="254" y="12.7" size="1.778" layer="97">Dickson charge pump
+<text x="254" y="10.16" size="1.778" layer="97">Dickson charge pump
 output: input + 5V
 freq:</text>
-<text x="254" y="7.62" size="1.778" layer="97">TODO: choose Schottky diodes</text>
 <text x="320.04" y="2.54" size="1.778" layer="97">power paths</text>
-<text x="137.16" y="10.16" size="1.778" layer="97">TODO: choose diodes (non Schottky)</text>
 <text x="391.16" y="2.54" size="1.778" layer="97">voltage monitoring paths
 4.9:1 divider</text>
@@
 <instance part="U3" gate="A" x="93.98" y="-55.88"/>
 <instance part="C3" gate="G$1" x="203.2" y="-10.16"/>
-<instance part="D4" gate="G$1" x="279.4" y="-2.54" smashed="yes">
-<attribute name="NAME" x="281.94" y="-2.0574" size="1.778" layer="95"/>
-</instance>
-<instance part="D6" gate="G$1" x="269.24" y="-2.54" smashed="yes">
-<attribute name="NAME" x="271.78" y="-2.0574" size="1.778" layer="95"/>
-</instance>
-<instance part="C5" gate="G$1" x="274.32" y="-7.62"/>
-<instance part="C6" gate="G$1" x="284.48" y="-7.62"/>
-<instance part="D7" gate="G$1" x="289.56" y="-2.54" smashed="yes">
-<attribute name="NAME" x="292.1" y="-2.0574" size="1.778" layer="95"/>
-</instance>
 <instance part="SUPPLY1" gate="GND" x="353.06" y="-38.1"/>
 <instance part="R1" gate="G$1" x="340.36" y="-71.12"/>
@@
 <attribute name="NAME" x="365.76" y="-60.96" size="1.778" layer="95"/>
 </instance>
-<instance part="T3" gate="G$1" x="350.52" y="-27.94"/>
-<instance part="T4" gate="G$1" x="350.52" y="-71.12"/>
-<instance part="C7" gate="G$1" x="294.64" y="-7.62"/>
+<instance part="T3" gate="G$1" x="350.52" y="-27.94" smashed="yes">
+<attribute name="NAME" x="355.6" y="-30.48" size="1.778" layer="95"/>
+<attribute name="VALUE" x="340.36" y="-22.86" size="1.778" layer="96"/>
+</instance>
+<instance part="T4" gate="G$1" x="350.52" y="-71.12" smashed="yes">
+<attribute name="NAME" x="355.6" y="-76.2" size="1.778" layer="95"/>
+<attribute name="VALUE" x="340.36" y="-66.04" size="1.778" layer="96"/>
+</instance>
 <instance part="C8" gate="A" x="241.3" y="2.54" smashed="yes" rot="R270">
 <attribute name="NAME" x="244.0686" y="0.9144" size="2.0828" layer="95" ratio="10" rot="SR0"/>
@@
 <instance part="D8" gate="G$1" x="152.4" y="-5.08"/>
 <instance part="D9" gate="G$1" x="200.66" y="10.16"/>
+<instance part="C4" gate="G$1" x="274.32" y="-7.62"/>
+<instance part="C5" gate="G$1" x="284.48" y="-7.62"/>
+<instance part="C6" gate="G$1" x="294.64" y="-7.62"/>
+<instance part="D1" gate="G$1" x="269.24" y="-2.54"/>
+<instance part="D2" gate="G$1" x="279.4" y="-2.54"/>
+<instance part="D3" gate="G$1" x="289.56" y="-2.54"/>
 </instances>
 <busses>
@@
 </segment>
 <segment>
-<pinref part="C7" gate="G$1" pin="-"/>
 <wire x1="294.64" y1="-12.7" x2="294.64" y2="-20.32" width="0.1524" layer="91"/>
 <wire x1="294.64" y1="-20.32" x2="254" y2="-20.32" width="0.1524" layer="91"/>
 <label x="254" y="-20.32" size="1.778" layer="95"/>
+<pinref part="C6" gate="G$1" pin="2"/>
 </segment>
 </net>
@@
 </segment>
 <segment>
-<pinref part="D6" gate="G$1" pin="A"/>
 <wire x1="266.7" y1="-2.54" x2="254" y2="-2.54" width="0.1524" layer="91"/>
 <label x="254" y="-2.54" size="1.778" layer="95"/>
+<pinref part="D1" gate="G$1" pin="A"/>
 </segment>
 </net>
@@
 <net name="N$4" class="0">
 <segment>
-<pinref part="D6" gate="G$1" pin="C"/>
-<pinref part="D4" gate="G$1" pin="A"/>
 <wire x1="271.78" y1="-2.54" x2="274.32" y2="-2.54" width="0.1524" layer="91"/>
-<pinref part="C5" gate="G$1" pin="+"/>
 <wire x1="274.32" y1="-2.54" x2="276.86" y2="-2.54" width="0.1524" layer="91"/>
 <wire x1="274.32" y1="-5.08" x2="274.32" y2="-2.54" width="0.1524" layer="91"/>
 <junction x="274.32" y="-2.54"/>
+<pinref part="C4" gate="G$1" pin="1"/>
+<pinref part="D1" gate="G$1" pin="C"/>
+<pinref part="D2" gate="G$1" pin="A"/>
 </segment>
 </net>
 <net name="N$5" class="0">
 <segment>
-<pinref part="D4" gate="G$1" pin="C"/>
 <wire x1="281.94" y1="-2.54" x2="284.48" y2="-2.54" width="0.1524" layer="91"/>
-<pinref part="C6" gate="G$1" pin="+"/>
 <wire x1="287.02" y1="-2.54" x2="284.48" y2="-2.54" width="0.1524" layer="91"/>
 <wire x1="284.48" y1="-2.54" x2="284.48" y2="-5.08" width="0.1524" layer="91"/>
-<pinref part="D7" gate="G$1" pin="A"/>
+<pinref part="C5" gate="G$1" pin="1"/>
+<pinref part="D2" gate="G$1" pin="C"/>
+<pinref part="D3" gate="G$1" pin="A"/>
 </segment>
 </net>
 <net name="PUMP_PWM#" class="0">
 <segment>
-<pinref part="C6" gate="G$1" pin="-"/>
 <wire x1="254" y1="-17.78" x2="284.48" y2="-17.78" width="0.1524" layer="91"/>
 <wire x1="284.48" y1="-17.78" x2="284.48" y2="-12.7" width="0.1524" layer="91"/>
 <label x="254" y="-17.78" size="1.778" layer="95"/>
+<pinref part="C5" gate="G$1" pin="2"/>
 </segment>
 <segment>
@@
 <net name="PUMP_V+" class="0">
 <segment>
-<pinref part="D7" gate="G$1" pin="C"/>
 <wire x1="292.1" y1="-2.54" x2="294.64" y2="-2.54" width="0.1524" layer="91"/>
 <label x="297.18" y="-2.54" size="1.778" layer="95"/>
-<pinref part="C7" gate="G$1" pin="+"/>
 <wire x1="294.64" y1="-2.54" x2="307.34" y2="-2.54" width="0.1524" layer="91"/>
 <wire x1="294.64" y1="-5.08" x2="294.64" y2="-2.54" width="0.1524" layer="91"/>
 <junction x="294.64" y="-2.54"/>
+<pinref part="C6" gate="G$1" pin="1"/>
+<pinref part="D3" gate="G$1" pin="C"/>
 </segment>
 <segment>
@@
 <net name="PUMP_PWM" class="0">
 <segment>
-<pinref part="C5" gate="G$1" pin="-"/>
 <wire x1="274.32" y1="-12.7" x2="274.32" y2="-15.24" width="0.1524" layer="91"/>
 <wire x1="274.32" y1="-15.24" x2="254" y2="-15.24" width="0.1524" layer="91"/>
 <label x="254" y="-15.24" size="1.778" layer="95"/>
-</segment>
-<segment>
+<pinref part="C4" gate="G$1" pin="2"/>
+</segment>
+<segment>

Commit message: routing
Parts:
- U$2: value TEENSY_3.0_ALLPINS -> TEENSY_3.0_BASIC-PGM; device Teensy3.0:TEENSY_3.0_ALLPINS -> Teensy3.0:TEENSY_3.0_BASIC-PGM
Changed lines of the file:
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@@
 <part name="R3" library="resistor" deviceset="R-US_" device="M0805" value="10K"/>
 <part name="SUPPLY2" library="supply2" deviceset="GND" device=""/>
-<part name="U$2" library="Teensy3.0" deviceset="TEENSY_3.0_ALLPINS" device=""/>
+<part name="U$2" library="Teensy3.0" deviceset="TEENSY_3.0_BASIC-PGM" device=""/>
 <part name="SPI_CON" library="pinhead" deviceset="PINHD-1X6" device=""/>
 <part name="R5" library="resistor" deviceset="R-US_" device="M0805" value="390K"/>
@@
 <instance part="R3" gate="G$1" x="353.06" y="-55.88" rot="R270"/>
 <instance part="SUPPLY2" gate="GND" x="353.06" y="-81.28"/>
-<instance part="U$2" gate="G$1" x="223.52" y="-68.58" smashed="yes">
-<attribute name="NAME" x="220.472" y="-34.29" size="1.27" layer="95" font="vector" ratio="15"/>
-<attribute name="VALUE" x="220.726" y="-106.68" size="1.27" layer="96" font="vector" ratio="15"/>
+<instance part="U$2" gate="G$1" x="223.52" y="-53.34" smashed="yes">
+<attribute name="NAME" x="220.472" y="-19.05" size="1.27" layer="95" font="vector" ratio="15"/>
+<attribute name="VALUE" x="213.106" y="-27.94" size="1.27" layer="96" font="vector" ratio="15"/>
 </instance>
 <instance part="SPI_CON" gate="A" x="43.18" y="-60.96" rot="MR0"/>
@@
 <segment>
 <pinref part="U$2" gate="G$1" pin="GND"/>
-<wire x1="238.76" y1="-48.26" x2="256.54" y2="-48.26" width="0.1524" layer="91"/>
-<label x="241.3" y="-48.26" size="1.778" layer="95"/>
+<wire x1="238.76" y1="-43.18" x2="256.54" y2="-43.18" width="0.1524" layer="91"/>
+<label x="238.76" y="-43.18" size="1.778" layer="95"/>
 </segment>
 <segment>
@@
 <segment>
 <pinref part="U$2" gate="G$1" pin="VIN"/>
-<wire x1="238.76" y1="-40.64" x2="256.54" y2="-40.64" width="0.1524" layer="91"/>
-<label x="241.3" y="-40.64" size="1.778" layer="95"/>
+<wire x1="238.76" y1="-38.1" x2="256.54" y2="-38.1" width="0.1524" layer="91"/>
+<label x="238.76" y="-38.1" size="1.778" layer="95"/>
 </segment>
 </net>
@@
 <segment>
 <pinref part="U$2" gate="G$1" pin="17/A3"/>
-<wire x1="238.76" y1="-93.98" x2="256.54" y2="-93.98" width="0.1524" layer="91"/>
-<label x="241.3" y="-93.98" size="1.778" layer="95"/>
+<wire x1="238.76" y1="-66.04" x2="256.54" y2="-66.04" width="0.1524" layer="91"/>
+<label x="238.76" y="-66.04" size="1.778" layer="95"/>
 </segment>
 </net>
@@
 <segment>
 <pinref part="U$2" gate="G$1" pin="3.3V"/>
-<wire x1="238.76" y1="-43.18" x2="256.54" y2="-43.18" width="0.1524" layer="91"/>
-<label x="241.3" y="-43.18" size="1.778" layer="95"/>
+<wire x1="238.76" y1="-40.64" x2="256.54" y2="-40.64" width="0.1524" layer="91"/>
+<label x="238.76" y="-40.64" size="1.778" layer="95"/>
 </segment>
 <segment>
@@
 <segment>
 <pinref part="U$2" gate="G$1" pin="14/A0"/>
-<wire x1="238.76" y1="-101.6" x2="256.54" y2="-101.6" width="0.1524" layer="91"/>
-<label x="241.3" y="-101.6" size="1.778" layer="95"/>
+<wire x1="238.76" y1="-73.66" x2="256.54" y2="-73.66" width="0.1524" layer="91"/>
+<label x="238.76" y="-73.66" size="1.778" layer="95"/>
 </segment>
 <segment>
@@
 <segment>
 <pinref part="U$2" gate="G$1" pin="16/A2"/>
-<wire x1="238.76" y1="-96.52" x2="256.54" y2="-96.52" width="0.1524" layer="91"/>
-<label x="241.3" y="-96.52" size="1.778" layer="95"/>
+<wire x1="238.76" y1="-68.58" x2="256.54" y2="-68.58" width="0.1524" layer="91"/>
+<label x="238.76" y="-68.58" size="1.778" layer="95"/>
 </segment>
 </net>
@@
 <segment>
 <pinref part="U$2" gate="G$1" pin="23/A9"/>
-<wire x1="238.76" y1="-78.74" x2="256.54" y2="-78.74" width="0.1524" layer="91"/>
-<label x="241.3" y="-78.74" size="1.778" layer="95"/>
+<wire x1="238.76" y1="-50.8" x2="256.54" y2="-50.8" width="0.1524" layer="91"/>
+<label x="238.76" y="-50.8" size="1.778" layer="95"/>
 </segment>
 <segment>
@@
 <segment>
 <pinref part="U$2" gate="G$1" pin="18/A4"/>
-<wire x1="238.76" y1="-91.44" x2="256.54" y2="-91.44" width="0.1524" layer="91"/>
-<label x="241.3" y="-91.44" size="1.778" layer="95"/>
+<wire x1="238.76" y1="-63.5" x2="256.54" y2="-63.5" width="0.1524" layer="91"/>
+<label x="238.76" y="-63.5" size="1.778" layer="95"/>
 </segment>
 </net>
@@
 <segment>
 <pinref part="U$2" gate="G$1" pin="19/A5"/>
-<wire x1="238.76" y1="-88.9" x2="256.54" y2="-88.9" width="0.1524" layer="91"/>
-<label x="241.3" y="-88.9" size="1.778" layer="95"/>
-</segment>
-</net>
+<wire x1="238.76" y1="-60.96" x2="256.54" y2="-60.96" width="0.1524" layer="91"/>
+<label x="238.76" y="-60.96" size="1.778" layer="95"/>
+</segment>
+</net>
