File: eagle/main.brd (EAGLE design)
At the start: 49.2 x 49.5 mm, 33 parts, among them IC1 TS5205, Q1 SI4840DY, Q5 SI4840DY, U1 SN74AHC1G00DCKR, U2 SN74AHC1G00DCKR, U3 SN74AHC1G00DCKR

Commit message: update
Parts:
- removed T1, T2: (no value), transistor:TO92
- added T3, T4: (no value), transistor:SOT23-BEC
- R1, R2, R3, R4, R6, R8: device resistor:0204V -> resistor:M0805
- R5, R7: value 400K -> 390K; device resistor:0204V -> resistor:M0805
- moved R3 93.2 mm to (19.1, 47.0)
- moved R8 91.1 mm to (19.1, 39.4)
- moved R7 87.2 mm to (24.1, 47.0)
- moved R6 82.5 mm to (24.1, 43.2)
- moved R5 78.4 mm to (24.1, 39.4)
- moved R2 74.1 mm to (29.2, 47.0)
- moved R1 69.9 mm to (29.2, 43.2)
- moved R4 51.3 mm to (19.1, 43.2)
- moved U$2 6.48 mm to (25.4, 19.1)
- moved Q5 1.27 mm to (11.4, 40.6)
Connections:
- net GND: now also T3.E, T4.E; no longer T1.1, T2.1
- net N$1: now also T3.C; no longer T1.3
- net N$2: now also T4.C; no longer T2.3
- net N$3: now also T4.B; no longer T2.2
- net N$6: now also T3.B; no longer T1.2

Commit message: update
Parts:
- removed C4: (no value), rcl:085CS_1AR
- added C7: 10u, rcl:085CS_1AR
- added C8: 100UF, Panasonic-EEEFK_EEEFP:CAPAE660X800N
- C1: value (none) -> 2.2u
- C5, C6: value (none) -> 10u
Connections:
- net GND: now also C7.-, C8.2; no longer C4.-
- net LOAD_V+: now also C8.1; no longer C4.+
- net PUMP_V+: now also C7.+
Changed lines of the file:
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@@
 <element name="D1" library="diode" package="DO35-7" value="1N4148DO35-7" x="-53.34" y="60.96"/>
 <element name="D2" library="diode" package="DO35-7" value="1N4148DO35-7" x="-71.12" y="60.96"/>
-<element name="C1" library="rcl" package="085CS_1AR" value="" x="-57.15" y="50.8"/>
+<element name="C1" library="rcl" package="085CS_1AR" value="2.2u" x="-57.15" y="50.8"/>
 <element name="R2" library="resistor" package="M0805" value="100K" x="29.21" y="46.99"/>
 <element name="R4" library="resistor" package="M0805" value="10K" x="19.05" y="43.18"/>
@@
 </element>
 <element name="C3" library="rcl" package="085CS_1AR" value="2.2u" x="-19.05" y="53.34"/>
-<element name="C4" library="rcl" package="085CS_1AR" value="" x="-68.58" y="50.8"/>
 <element name="D4" library="diode" package="DO35-7" value="1N4148DO35-7" x="-41.91" y="68.58"/>
 <element name="D6" library="diode" package="DO35-7" value="1N4148DO35-7" x="-59.69" y="68.58"/>
-<element name="C5" library="rcl" package="085CS_1AR" value="" x="-19.05" y="60.96"/>
-<element name="C6" library="rcl" package="085CS_1AR" value="" x="-30.48" y="60.96"/>
+<element name="C5" library="rcl" package="085CS_1AR" value="10u" x="-19.05" y="60.96"/>
+<element name="C6" library="rcl" package="085CS_1AR" value="10u" x="-30.48" y="60.96"/>
 <element name="D7" library="diode" package="DO35-7" value="1N4148DO35-7" x="-24.13" y="74.93"/>
 <element name="R1" library="resistor" package="M0805" value="100K" x="29.21" y="43.18"/>
@@
 <element name="T3" library="transistor" package="SOT23-BEC" value="" x="-73.66" y="-3.81"/>
 <element name="T4" library="transistor" package="SOT23-BEC" value="" x="-73.66" y="-10.16"/>
+<element name="C7" library="rcl" package="085CS_1AR" value="10u" x="-71.12" y="-16.51"/>
+<element name="C8" library="Panasonic-EEEFK_EEEFP" package="CAPAE660X800N" value="100UF" x="43.18" y="27.94">
+<attribute name="PACKAGE" value="CASE-D8" x="43.18" y="27.94" size="1.778" layer="27" display="off"/>
+<attribute name="OC_NEWARK" value="23T0852" x="43.18" y="27.94" size="1.778" layer="27" display="off"/>
+<attribute name="TOLERANCE" value="±20 %" x="43.18" y="27.94" size="1.778" layer="27" display="off"/>
+<attribute name="MPN" value="EEE-FK1E101XP" x="43.18" y="27.94" size="1.778" layer="27" display="off"/>
+<attribute name="SUPPLIER" value="PANASONIC" x="43.18" y="27.94" size="1.778" layer="27" display="off"/>
+<attribute name="VOLTAGERATING" value="25V" x="43.18" y="27.94" size="1.778" layer="27" display="off"/>
+<attribute name="OC_FARNELL" value="1850109  " x="43.18" y="27.94" size="1.778" layer="27" display="off"/>
+</element>
 </elements>
 <signals>
@@
 <contactref element="U2" pad="3"/>
 <contactref element="U3" pad="3"/>
-<contactref element="C4" pad="-"/>
 <contactref element="U$2" pad="GND"/>
 <contactref element="U$2" pad="GND1"/>
@@
 <contactref element="T3" pad="E"/>
 <contactref element="T4" pad="E"/>
+<contactref element="C7" pad="-"/>
+<contactref element="C8" pad="2"/>
+<wire x1="-74.37" y1="-16.51" x2="45.593" y2="27.94" width="0" layer="19" extent="1-1"/>
+<wire x1="-72.71" y1="-11.26" x2="-74.37" y2="-16.51" width="0" layer="19" extent="1-1"/>
 <wire x1="-72.71" y1="-4.91" x2="-72.71" y2="-11.26" width="0" layer="19" extent="1-1"/>
 <wire x1="-68.3514" y1="5.6896" x2="-72.71" y2="-4.91" width="0" layer="19" extent="1-1"/>
 <wire x1="-73.4314" y1="42.5196" x2="-68.3514" y2="5.6896" width="0" layer="19" extent="1-1"/>
-<wire x1="-71.83" y1="50.8" x2="-73.4314" y2="42.5196" width="0" layer="19" extent="1-1"/>
-<wire x1="-60.4" y1="50.8" x2="-71.83" y2="50.8" width="0" layer="19" extent="1-1"/>
+<wire x1="-60.4" y1="50.8" x2="-73.4314" y2="42.5196" width="0" layer="19" extent="1-1"/>
 <wire x1="-48.26" y1="52.04" x2="-60.4" y2="50.8" width="0" layer="19" extent="1-1"/>
 <wire x1="-41.6814" y1="42.5196" x2="-48.26" y2="52.04" width="0" layer="19" extent="1-1"/>
 <wire x1="-38.1" y1="60.96" x2="-48.26" y2="52.04" width="0" layer="19" extent="1-1"/>
 <wire x1="-22.3" y1="53.34" x2="-38.1" y2="60.96" width="0" layer="19" extent="1-1"/>
-<wire x1="25.08" y1="43.18" x2="-38.1" y2="60.96" width="0" layer="19" extent="1-1"/>
-<wire x1="-53.34" y1="80.01" x2="25.08" y2="43.18" width="0" layer="19" extent="1-1"/>
-<wire x1="-41.91" y1="80.01" x2="25.08" y2="43.18" width="0" layer="19" extent="1-1"/>
+<wire x1="-41.91" y1="80.01" x2="-38.1" y2="60.96" width="0" layer="19" extent="1-1"/>
 <wire x1="-33.02" y1="80.01" x2="-41.91" y2="80.01" width="0" layer="19" extent="1-1"/>
+<wire x1="-53.34" y1="80.01" x2="-41.91" y2="80.01" width="0" layer="19" extent="1-1"/>
 <wire x1="-64.77" y1="80.01" x2="-53.34" y2="80.01" width="0" layer="19" extent="1-1"/>
 <wire x1="17.78" y1="35.56" x2="-22.3" y2="53.34" width="0" layer="19" extent="1-1"/>
 <wire x1="20" y1="39.37" x2="17.78" y2="35.56" width="0" layer="19" extent="1-1"/>
+<wire x1="25.08" y1="43.18" x2="20" y2="39.37" width="0" layer="19" extent="1-1"/>
 <wire x1="25.4" y1="17.78" x2="17.78" y2="35.56" width="0" layer="19" extent="1-1"/>
 <wire x1="25.4" y1="2.54" x2="25.4" y2="17.78" width="0" layer="19" extent="1-1"/>
@@
 <signal name="LOAD_V+">
 <contactref element="LOAD_CON" pad="1"/>
-<contactref element="C4" pad="+"/>
 <contactref element="Q5" pad="1-3"/>
 <contactref element="Q1" pad="1-3"/>
-<wire x1="10.795" y1="38.04" x2="38.735" y2="38.04" width="0" layer="19" extent="1-1"/>
-<wire x1="-65.33" y1="50.8" x2="10.795" y2="38.04" width="0" layer="19" extent="1-1"/>
-<wire x1="-67.31" y1="80.01" x2="-65.33" y2="50.8" width="0" layer="19" extent="1-1"/>
+<contactref element="C8" pad="1"/>
+<wire x1="10.795" y1="38.04" x2="40.767" y2="27.94" width="0" layer="19" extent="1-1"/>
+<wire x1="38.735" y1="38.04" x2="10.795" y2="38.04" width="0" layer="19" extent="1-1"/>
+<wire x1="-67.31" y1="80.01" x2="10.795" y2="38.04" width="0" layer="19" extent="1-1"/>
 </signal>
 <signal name="N$4">
@@
 <contactref element="R4" pad="1"/>
 <contactref element="R3" pad="1"/>
-<wire x1="-27.94" y1="74.93" x2="18.1" y2="43.18" width="0" layer="19" extent="1-1"/>
+<contactref element="C7" pad="+"/>
+<wire x1="-27.94" y1="74.93" x2="-67.87" y2="-16.51" width="0" layer="19" extent="1-1"/>
 <wire x1="18.1" y1="46.99" x2="-27.94" y2="74.93" width="0" layer="19" extent="1-1"/>
+<wire x1="18.1" y1="43.18" x2="18.1" y2="46.99" width="0" layer="19" extent="1-1"/>
 </signal>
 <signal name="N$1">

Commit message: update
Parts:
- C1, C3: device rcl:085CS_1AR -> rcl:C1210K
- C2: device resistor:C025-024X044 -> rcl:C0805K
Connections:
- net GND: now also C1.2, C3.2; no longer C1.-, C3.-
- net LOGIC_V+: now also C3.1; no longer C3.+
- net POW01_V+: now also C1.1; no longer C1.+
Changed lines of the file:
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@@
 <element name="D1" library="diode" package="DO35-7" value="1N4148DO35-7" x="-53.34" y="60.96"/>
 <element name="D2" library="diode" package="DO35-7" value="1N4148DO35-7" x="-71.12" y="60.96"/>
-<element name="C1" library="rcl" package="085CS_1AR" value="2.2u" x="-57.15" y="50.8"/>
+<element name="C1" library="rcl" package="C1210K" value="2.2u" x="-57.15" y="50.8"/>
 <element name="R2" library="resistor" package="M0805" value="100K" x="29.21" y="46.99"/>
 <element name="R4" library="resistor" package="M0805" value="10K" x="19.05" y="43.18"/>
@@
 <attribute name="OC_FARNELL" value="1287496" x="0" y="0" size="1.778" layer="27" display="off"/>
 </element>
-<element name="C3" library="rcl" package="085CS_1AR" value="2.2u" x="-19.05" y="53.34"/>
+<element name="C3" library="rcl" package="C1210K" value="2.2u" x="-19.05" y="53.34"/>
 <element name="D4" library="diode" package="DO35-7" value="1N4148DO35-7" x="-41.91" y="68.58"/>
 <element name="D6" library="diode" package="DO35-7" value="1N4148DO35-7" x="-59.69" y="68.58"/>
@@
 <element name="R8" library="resistor" package="M0805" value="100K" x="19.05" y="39.37"/>
 <element name="IC1" library="v-reg" package="SOT25" value="TS5205" x="-48.26" y="53.34"/>
-<element name="C2" library="resistor" package="C025-024X044" value="470p" x="-39.37" y="60.96"/>
+<element name="C2" library="rcl" package="C0805K" value="470p" x="-39.37" y="60.96"/>
 <element name="Q5" library="transistor-fet" package="SO08-E3" value="SI4840DY" x="11.43" y="40.64"/>
 <element name="Q1" library="transistor-fet" package="SO08-E3" value="SI4840DY" x="39.37" y="40.64"/>
@@
 <contactref element="POW1_CON" pad="2"/>
 <contactref element="LOAD_CON" pad="2"/>
-<contactref element="C1" pad="-"/>
+<contactref element="C1" pad="2"/>
 <contactref element="IC1" pad="2"/>
-<contactref element="C3" pad="-"/>
+<contactref element="C3" pad="2"/>
 <contactref element="C2" pad="2"/>
 <contactref element="U1" pad="3"/>
@@
 <wire x1="-68.3514" y1="5.6896" x2="-72.71" y2="-4.91" width="0" layer="19" extent="1-1"/>
 <wire x1="-73.4314" y1="42.5196" x2="-68.3514" y2="5.6896" width="0" layer="19" extent="1-1"/>
-<wire x1="-60.4" y1="50.8" x2="-73.4314" y2="42.5196" width="0" layer="19" extent="1-1"/>
-<wire x1="-48.26" y1="52.04" x2="-60.4" y2="50.8" width="0" layer="19" extent="1-1"/>
+<wire x1="-55.65" y1="50.8" x2="-73.4314" y2="42.5196" width="0" layer="19" extent="1-1"/>
+<wire x1="-48.26" y1="52.04" x2="-55.65" y2="50.8" width="0" layer="19" extent="1-1"/>
 <wire x1="-41.6814" y1="42.5196" x2="-48.26" y2="52.04" width="0" layer="19" extent="1-1"/>
-<wire x1="-38.1" y1="60.96" x2="-48.26" y2="52.04" width="0" layer="19" extent="1-1"/>
-<wire x1="-22.3" y1="53.34" x2="-38.1" y2="60.96" width="0" layer="19" extent="1-1"/>
-<wire x1="-41.91" y1="80.01" x2="-38.1" y2="60.96" width="0" layer="19" extent="1-1"/>
+<wire x1="-38.37" y1="60.96" x2="-48.26" y2="52.04" width="0" layer="19" extent="1-1"/>
+<wire x1="-17.55" y1="53.34" x2="-38.37" y2="60.96" width="0" layer="19" extent="1-1"/>
+<wire x1="-41.91" y1="80.01" x2="-38.37" y2="60.96" width="0" layer="19" extent="1-1"/>
 <wire x1="-33.02" y1="80.01" x2="-41.91" y2="80.01" width="0" layer="19" extent="1-1"/>
 <wire x1="-53.34" y1="80.01" x2="-41.91" y2="80.01" width="0" layer="19" extent="1-1"/>
 <wire x1="-64.77" y1="80.01" x2="-53.34" y2="80.01" width="0" layer="19" extent="1-1"/>
-<wire x1="17.78" y1="35.56" x2="-22.3" y2="53.34" width="0" layer="19" extent="1-1"/>
+<wire x1="17.78" y1="35.56" x2="-17.55" y2="53.34" width="0" layer="19" extent="1-1"/>
 <wire x1="20" y1="39.37" x2="17.78" y2="35.56" width="0" layer="19" extent="1-1"/>
 <wire x1="25.08" y1="43.18" x2="20" y2="39.37" width="0" layer="19" extent="1-1"/>
@@
 <contactref element="D1" pad="C"/>
 <contactref element="D2" pad="C"/>
-<contactref element="C1" pad="+"/>
+<contactref element="C1" pad="1"/>
 <contactref element="IC1" pad="1"/>
 <contactref element="IC1" pad="3"/>
@@
 <wire x1="-57.15" y1="60.96" x2="-74.93" y2="60.96" width="0" layer="19" extent="1-1"/>
 <wire x1="-55.88" y1="68.58" x2="-57.15" y2="60.96" width="0" layer="19" extent="1-1"/>
-<wire x1="-53.9" y1="50.8" x2="-57.15" y2="60.96" width="0" layer="19" extent="1-1"/>
-<wire x1="-49.21" y1="52.04" x2="-53.9" y2="50.8" width="0" layer="19" extent="1-1"/>
+<wire x1="-58.65" y1="50.8" x2="-57.15" y2="60.96" width="0" layer="19" extent="1-1"/>
+<wire x1="-49.21" y1="52.04" x2="-58.65" y2="50.8" width="0" layer="19" extent="1-1"/>
 <wire x1="-47.31" y1="52.04" x2="-49.21" y2="52.04" width="0" layer="19" extent="1-1"/>
 </signal>
@@
 <contactref element="D3" pad="A"/>
 <contactref element="IC1" pad="5"/>
-<contactref element="C3" pad="+"/>
+<contactref element="C3" pad="1"/>
 <contactref element="U$2" pad="VIN"/>
-<wire x1="-15.8" y1="53.34" x2="-20.32" y2="68.58" width="0" layer="19" extent="1-1"/>
-<wire x1="33.02" y1="35.56" x2="-15.8" y2="53.34" width="0" layer="19" extent="1-1"/>
+<wire x1="-20.55" y1="53.34" x2="-20.32" y2="68.58" width="0" layer="19" extent="1-1"/>
+<wire x1="33.02" y1="35.56" x2="-20.55" y2="53.34" width="0" layer="19" extent="1-1"/>
 <wire x1="-49.21" y1="54.64" x2="-20.32" y2="68.58" width="0" layer="19" extent="1-1"/>
 </signal>
@@
 <contactref element="IC1" pad="4"/>
 <contactref element="C2" pad="1"/>
-<wire x1="-47.31" y1="54.64" x2="-40.64" y2="60.96" width="0" layer="19" extent="1-1"/>
+<wire x1="-47.31" y1="54.64" x2="-40.37" y2="60.96" width="0" layer="19" extent="1-1"/>
 </signal>
 <signal name="MCU_ADC0">

Commit message: schottky diodes
Parts:
- removed D1, D2, D3: 1N4148DO35-7, diode:DO35-7
- added D5, D8, D9: (no value), diode:DO214AC
- C1, C3: value 2.2u -> 4.7u
- moved IC1 57.4 mm to (3.81, 29.2)
Connections:
- net LOGIC_V+: now also D9.A; no longer D3.A
- net POW01_V+: now also D5.C, D8.C; no longer D1.C, D2.C
- net POW0_V+: now also D5.A; no longer D1.A
- net POW1_V+: now also D8.A; no longer D2.A
- net SPI_V+: now also D9.C; no longer D3.C
Changed lines of the file:
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@@
 <element name="POW1_CON" library="pinhead" package="1X02" value="" x="-54.61" y="80.01"/>
 <element name="LOAD_CON" library="pinhead" package="1X02" value="" x="-66.04" y="80.01"/>
-<element name="D1" library="diode" package="DO35-7" value="1N4148DO35-7" x="-53.34" y="60.96"/>
-<element name="D2" library="diode" package="DO35-7" value="1N4148DO35-7" x="-71.12" y="60.96"/>
-<element name="C1" library="rcl" package="C1210K" value="2.2u" x="-57.15" y="50.8"/>
+<element name="C1" library="rcl" package="C1210K" value="4.7u" x="-57.15" y="50.8"/>
 <element name="R2" library="resistor" package="M0805" value="100K" x="29.21" y="46.99"/>
 <element name="R4" library="resistor" package="M0805" value="10K" x="19.05" y="43.18"/>
@@
 <attribute name="OC_FARNELL" value="1287496" x="0" y="0" size="1.778" layer="27" display="off"/>
 </element>
-<element name="C3" library="rcl" package="C1210K" value="2.2u" x="-19.05" y="53.34"/>
+<element name="C3" library="rcl" package="C1210K" value="4.7u" x="-19.05" y="53.34"/>
 <element name="D4" library="diode" package="DO35-7" value="1N4148DO35-7" x="-41.91" y="68.58"/>
 <element name="D6" library="diode" package="DO35-7" value="1N4148DO35-7" x="-59.69" y="68.58"/>
@@
 <element name="R3" library="resistor" package="M0805" value="10K" x="19.05" y="46.99"/>
 <element name="U$2" library="Teensy3.0" package="TEENSY_3.0_ALLPINS" value="TEENSY_3.0_ALLPINS" x="25.4" y="19.05"/>
-<element name="D3" library="diode" package="DO35-7" value="1N4148DO35-7" x="-24.13" y="68.58"/>
 <element name="SPI_CON" library="pinhead" package="1X06" value="" x="-26.67" y="80.01"/>
 <element name="R5" library="resistor" package="M0805" value="390K" x="24.13" y="39.37"/>
@@
 <element name="R7" library="resistor" package="M0805" value="390K" x="24.13" y="46.99"/>
 <element name="R8" library="resistor" package="M0805" value="100K" x="19.05" y="39.37"/>
-<element name="IC1" library="v-reg" package="SOT25" value="TS5205" x="-48.26" y="53.34"/>
+<element name="IC1" library="v-reg" package="SOT25" value="TS5205" x="3.81" y="29.21"/>
 <element name="C2" library="rcl" package="C0805K" value="470p" x="-39.37" y="60.96"/>
 <element name="Q5" library="transistor-fet" package="SO08-E3" value="SI4840DY" x="11.43" y="40.64"/>
@@
 <attribute name="OC_FARNELL" value="1850109  " x="43.18" y="27.94" size="1.778" layer="27" display="off"/>
 </element>
+<element name="D5" library="diode" package="DO214AC" value="" x="-73.66" y="-24.13"/>
+<element name="D8" library="diode" package="DO214AC" value="" x="-73.66" y="-29.21"/>
+<element name="D9" library="diode" package="DO214AC" value="" x="-73.66" y="-34.29"/>
 </elements>
 <signals>
@@
 <signal name="POW0_V+">
 <contactref element="POW0_CON" pad="1"/>
-<contactref element="D1" pad="A"/>
 <contactref element="Q5" pad="5-8"/>
 <contactref element="R5" pad="1"/>
-<wire x1="23.18" y1="39.37" x2="-44.45" y2="80.01" width="0" layer="19" extent="1-1"/>
-<wire x1="-49.53" y1="60.96" x2="23.18" y2="39.37" width="0" layer="19" extent="1-1"/>
-<wire x1="11.43" y1="43.24" x2="-49.53" y2="60.96" width="0" layer="19" extent="1-1"/>
+<contactref element="D5" pad="A"/>
+<wire x1="11.43" y1="43.24" x2="-71.61" y2="-24.13" width="0" layer="19" extent="1-1"/>
+<wire x1="23.18" y1="39.37" x2="11.43" y2="43.24" width="0" layer="19" extent="1-1"/>
+<wire x1="-44.45" y1="80.01" x2="11.43" y2="43.24" width="0" layer="19" extent="1-1"/>
 </signal>
 <signal name="GND">
@@
 <wire x1="-73.4314" y1="42.5196" x2="-68.3514" y2="5.6896" width="0" layer="19" extent="1-1"/>
 <wire x1="-55.65" y1="50.8" x2="-73.4314" y2="42.5196" width="0" layer="19" extent="1-1"/>
-<wire x1="-48.26" y1="52.04" x2="-55.65" y2="50.8" width="0" layer="19" extent="1-1"/>
-<wire x1="-41.6814" y1="42.5196" x2="-48.26" y2="52.04" width="0" layer="19" extent="1-1"/>
-<wire x1="-38.37" y1="60.96" x2="-48.26" y2="52.04" width="0" layer="19" extent="1-1"/>
+<wire x1="3.81" y1="27.91" x2="-55.65" y2="50.8" width="0" layer="19" extent="1-1"/>
+<wire x1="-41.6814" y1="42.5196" x2="3.81" y2="27.91" width="0" layer="19" extent="1-1"/>
+<wire x1="-38.37" y1="60.96" x2="3.81" y2="27.91" width="0" layer="19" extent="1-1"/>
 <wire x1="-17.55" y1="53.34" x2="-38.37" y2="60.96" width="0" layer="19" extent="1-1"/>
 <wire x1="-41.91" y1="80.01" x2="-38.37" y2="60.96" width="0" layer="19" extent="1-1"/>
@@
 </signal>
 <signal name="POW01_V+">
-<contactref element="D1" pad="C"/>
-<contactref element="D2" pad="C"/>
 <contactref element="C1" pad="1"/>
 <contactref element="IC1" pad="1"/>
 <contactref element="IC1" pad="3"/>
 <contactref element="D6" pad="A"/>
-<wire x1="-57.15" y1="60.96" x2="-74.93" y2="60.96" width="0" layer="19" extent="1-1"/>
-<wire x1="-55.88" y1="68.58" x2="-57.15" y2="60.96" width="0" layer="19" extent="1-1"/>
-<wire x1="-58.65" y1="50.8" x2="-57.15" y2="60.96" width="0" layer="19" extent="1-1"/>
-<wire x1="-49.21" y1="52.04" x2="-58.65" y2="50.8" width="0" layer="19" extent="1-1"/>
-<wire x1="-47.31" y1="52.04" x2="-49.21" y2="52.04" width="0" layer="19" extent="1-1"/>
+<contactref element="D5" pad="C"/>
+<contactref element="D8" pad="C"/>
+<wire x1="-75.71" y1="-24.13" x2="-75.71" y2="-29.21" width="0" layer="19" extent="1-1"/>
+<wire x1="-58.65" y1="50.8" x2="-75.71" y2="-24.13" width="0" layer="19" extent="1-1"/>
+<wire x1="-55.88" y1="68.58" x2="-58.65" y2="50.8" width="0" layer="19" extent="1-1"/>
+<wire x1="2.86" y1="27.91" x2="-58.65" y2="50.8" width="0" layer="19" extent="1-1"/>
+<wire x1="4.76" y1="27.91" x2="2.86" y2="27.91" width="0" layer="19" extent="1-1"/>
 </signal>
 <signal name="LOGIC_V+">
-<contactref element="D3" pad="A"/>
 <contactref element="IC1" pad="5"/>
 <contactref element="C3" pad="1"/>
 <contactref element="U$2" pad="VIN"/>
-<wire x1="-20.55" y1="53.34" x2="-20.32" y2="68.58" width="0" layer="19" extent="1-1"/>
-<wire x1="33.02" y1="35.56" x2="-20.55" y2="53.34" width="0" layer="19" extent="1-1"/>
-<wire x1="-49.21" y1="54.64" x2="-20.32" y2="68.58" width="0" layer="19" extent="1-1"/>
+<contactref element="D9" pad="A"/>
+<wire x1="2.86" y1="30.51" x2="-71.61" y2="-34.29" width="0" layer="19" extent="1-1"/>
+<wire x1="33.02" y1="35.56" x2="2.86" y2="30.51" width="0" layer="19" extent="1-1"/>
+<wire x1="-20.55" y1="53.34" x2="2.86" y2="30.51" width="0" layer="19" extent="1-1"/>
 </signal>
 <signal name="XCOND_EN">
@@
 <signal name="POW1_V+">
 <contactref element="POW1_CON" pad="1"/>
-<contactref element="D2" pad="A"/>
 <contactref element="Q1" pad="5-8"/>
 <contactref element="R7" pad="1"/>
-<wire x1="23.18" y1="46.99" x2="39.37" y2="43.24" width="0" layer="19" extent="1-1"/>
-<wire x1="-55.88" y1="80.01" x2="23.18" y2="46.99" width="0" layer="19" extent="1-1"/>
-<wire x1="-67.31" y1="60.96" x2="23.18" y2="46.99" width="0" layer="19" extent="1-1"/>
+<contactref element="D8" pad="A"/>
+<wire x1="-55.88" y1="80.01" x2="-71.61" y2="-29.21" width="0" layer="19" extent="1-1"/>
+<wire x1="23.18" y1="46.99" x2="-55.88" y2="80.01" width="0" layer="19" extent="1-1"/>
+<wire x1="39.37" y1="43.24" x2="23.18" y2="46.99" width="0" layer="19" extent="1-1"/>
 </signal>
 <signal name="LOAD_V+">
@@
 </signal>
 <signal name="SPI_V+">
-<contactref element="D3" pad="C"/>
 <contactref element="SPI_CON" pad="6"/>
-<wire x1="-27.94" y1="68.58" x2="-20.32" y2="80.01" width="0" layer="19" extent="1-1"/>
+<contactref element="D9" pad="C"/>
+<wire x1="-20.32" y1="80.01" x2="-75.71" y2="-34.29" width="0" layer="19" extent="1-1"/>
 </signal>
 <signal name="SPI_CS">
@@
 <contactref element="IC1" pad="4"/>
 <contactref element="C2" pad="1"/>
-<wire x1="-47.31" y1="54.64" x2="-40.37" y2="60.96" width="0" layer="19" extent="1-1"/>
+<wire x1="4.76" y1="30.51" x2="-40.37" y2="60.96" width="0" layer="19" extent="1-1"/>
 </signal>
 <signal name="MCU_ADC0">

Commit message: update board
Parts:
- removed C7: 10u, rcl:085CS_1AR
- removed D4, D6, D7: 1N4148DO35-7, diode:DO35-7
- added C4: 4.7u, rcl:C1210K
- added D1, D2, D3: (no value), diode:DO214AC
- C5, C6: value 10u -> 4.7u; device rcl:085CS_1AR -> rcl:C1210K
- moved LOAD_CON 118.2 mm to (41.9, 31.8)
- moved T4 112.6 mm to (36.8, 11.4), turned to 270 degrees
- moved T3 110.8 mm to (36.8, 3.81), turned to 270 degrees
- moved U3 101.2 mm to (24.1, 12.7)
- moved POW1_CON 96.0 mm to (35.6, 47.0)
- moved D9 95.4 mm to (11.4, 8.89)
- moved U1 91.4 mm to (24.1, 7.62)
- moved POW0_CON 91.3 mm to (41.9, 47.0), turned to 180 degrees
- moved D8 88.1 mm to (3.81, 12.7)
- moved D5 84.7 mm to (3.81, 10.2)
- moved U2 76.5 mm to (24.1, 2.54)
- moved C1 75.4 mm to (3.81, 6.35)
- moved C2 74.6 mm to (11.4, 6.35)
- moved C6 59.3 mm to (11.4, 19.1)
- moved SPI_CON 51.4 mm to (12.7, 47.0), turned to 180 degrees
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Connections:
- net GND: now also C6.2; no longer C7.-
- net N$4: now also C4.1, D1.C, D2.A; no longer C5.+, D4.A, D6.C
- net N$5: now also C5.1, D2.C, D3.A; no longer C6.+, D4.C, D7.A
- net POW01_V+: now also D1.A; no longer D6.A
- net PUMP_PWM: now also C4.2; no longer C5.-
- net PUMP_PWM#: now also C5.2; no longer C6.-
- net PUMP_V+: now also C6.1, D3.C; no longer C7.+, D7.C
Routing:
- added copper zone on layer 1, net GND
- added copper zone on layer 16, net GND
