File: eagle/main.brd (EAGLE design)
At the start: 49.2 x 49.5 mm, 34 parts, among them IC1 TS5205, Q1 SI4840DY, Q5 SI4840DY, U1 SN74AHC1G00DCKR, U2 SN74AHC1G00DCKR, U3 SN74AHC1G00DCKR

Commit message: routing
Parts:
- U$2: value TEENSY_3.0_ALLPINS -> TEENSY_3.0_BASIC-PGM; device Teensy3.0:TEENSY_3.0_ALLPINS -> Teensy3.0:TEENSY_3.0_BASIC-PGM
- moved D9 33.1 mm to (8.89, 41.9), turned to 270 degrees
- moved U2 22.2 mm to (45.7, 7.62), flipped to the bottom, turned to 180 degrees
- moved R2 19.9 mm to (47.0, 11.4), flipped to the bottom, turned to 90 degrees
- moved D5 19.7 mm to (23.5, 8.89)
- moved D8 19.7 mm to (23.5, 12.7)
- moved U1 17.8 mm to (41.9, 7.62), flipped to the bottom, turned to 90 degrees
- moved R4 16.5 mm to (44.5, 11.4), flipped to the bottom, turned to 90 degrees
- moved T3 15.5 mm to (45.7, 16.5), flipped to the bottom, turned to 0 degrees
- moved U3 14.9 mm to (38.1, 7.62), flipped to the bottom, turned to 180 degrees
- moved IC1 10.5 mm to (11.4, 12.7), turned to 270 degrees
- moved R1 10.2 mm to (39.4, 11.4), flipped to the bottom, turned to 90 degrees
- moved C1 7.73 mm to (11.4, 5.08)
- moved R3 7.73 mm to (36.8, 11.4), flipped to the bottom, turned to 90 degrees
- moved C3 6.35 mm to (5.08, 12.7), turned to 180 degrees
- moved T4 5.24 mm to (38.1, 16.5), flipped to the bottom, turned to 0 degrees
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Connections:
- removed net AREF: U$2.AREF
- removed net VUSB: U$2.VUSB
- net GND: no longer U$2.GND2
- net MCU_V+: no longer U$2.3.3V2
Routing:
- net N$1: track 0.00 -> 35.6 mm, vias 0 -> 1
- net N$2: track 0.00 -> 35.6 mm, vias 0 -> 1
- net LOAD_V+: track 0.00 -> 27.9 mm
- net POW0_EN: track 0.00 -> 15.1 mm
- net POW1_EN: track 0.00 -> 11.7 mm
- net XCOND_EN: track 0.00 -> 8.66 mm
- net POW1_V+: track 0.00 -> 6.41 mm
- net POW0_V+: track 0.00 -> 6.41 mm
- net PUMP_PWM#: track 0.00 -> 6.12 mm
- net PUMP_PWM: track 0.00 -> 6.12 mm
- net N$6: track 0.00 -> 3.35 mm
- net N$3: track 0.00 -> 3.35 mm
- net POW1_DIS: track 0.00 -> 2.43 mm
- net POW0_DIS: track 0.00 -> 2.43 mm

Commit message: update routing
Parts:
- moved C1 8.82 mm to (6.99, 12.7), turned to 180 degrees
- moved C3 6.63 mm to (6.99, 6.35)
- moved C6 4.62 mm to (6.99, 18.4), turned to 90 degrees
- moved C2 4.49 mm to (6.99, 9.53)
- moved IC1 1.42 mm to (12.1, 11.4), turned to 180 degrees
- turned D1 to 270 degrees
Routing:
- net POW0_VMON: track 0.00 -> 29.5 mm
- net POW1_VMON: track 0.00 -> 27.9 mm
- net N$4: track 0.00 -> 6.90 mm
- net PUMP_V+: track 0.00 -> 4.59 mm
- net N$5: track 0.00 -> 4.15 mm
- net SPI_V+: track 0.00 -> 3.03 mm
Changed lines of the file:
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@@
 <element name="POW1_CON" library="pinhead" package="1X02" value="" x="38.1" y="46.99"/>
 <element name="LOAD_CON" library="pinhead" package="1X02" value="" x="41.91" y="31.75" rot="R270"/>
-<element name="C1" library="rcl" package="C1210K" value="4.7u" x="11.43" y="5.08"/>
+<element name="C1" library="rcl" package="C1210K" value="4.7u" x="6.985" y="12.7" rot="R180"/>
 <element name="R2" library="resistor" package="M0805" value="100K" x="46.99" y="11.43" rot="MR90"/>
 <element name="R4" library="resistor" package="M0805" value="10K" x="44.45" y="11.43" rot="MR90"/>
@@
 <attribute name="OC_FARNELL" value="1287496" x="110.49" y="50.8" size="1.778" layer="28" rot="MR180" display="off"/>
 </element>
-<element name="C3" library="rcl" package="C1210K" value="4.7u" x="5.08" y="12.7" rot="R180"/>
+<element name="C3" library="rcl" package="C1210K" value="4.7u" x="6.985" y="6.35" rot="R180"/>
 <element name="R1" library="resistor" package="M0805" value="100K" x="39.37" y="11.43" rot="MR90"/>
 <element name="R3" library="resistor" package="M0805" value="10K" x="36.83" y="11.43" rot="MR90"/>
@@
 <element name="R7" library="resistor" package="M0805" value="390K" x="29.21" y="26.67" rot="R270"/>
 <element name="R8" library="resistor" package="M0805" value="100K" x="29.21" y="31.75" rot="R270"/>
-<element name="IC1" library="v-reg" package="SOT25" value="TS5205" x="11.43" y="12.7" rot="R270"/>
-<element name="C2" library="rcl" package="C0805K" value="470p" x="11.43" y="8.89" rot="R180"/>
+<element name="IC1" library="v-reg" package="SOT25" value="TS5205" x="12.065" y="11.43" rot="R180"/>
+<element name="C2" library="rcl" package="C0805K" value="470p" x="6.985" y="9.525" rot="R180"/>
 <element name="Q5" library="transistor-fet" package="SO08-E3" value="SI4840DY" x="45.72" y="39.37"/>
 <element name="Q1" library="transistor-fet" package="SO08-E3" value="SI4840DY" x="38.1" y="39.37"/>
@@
 <element name="C4" library="rcl" package="C1210K" value="4.7u" x="11.43" y="29.21"/>
 <element name="C5" library="rcl" package="C1210K" value="4.7u" x="11.43" y="24.13"/>
-<element name="C6" library="rcl" package="C1210K" value="4.7u" x="11.43" y="17.145"/>
-<element name="D1" library="diode" package="DO214AC" value="" x="6.985" y="27.305" rot="R90"/>
+<element name="C6" library="rcl" package="C1210K" value="4.7u" x="6.985" y="18.415" rot="R90"/>
+<element name="D1" library="diode" package="DO214AC" value="" x="6.985" y="27.305" rot="R270"/>
 <element name="D2" library="diode" package="DO214AC" value="" x="3.175" y="27.305" rot="R90"/>
 <element name="D3" library="diode" package="DO214AC" value="" x="3.175" y="19.05" rot="R90"/>
@@
 <contactref element="D1" pad="A"/>
 <wire x1="21.445" y1="8.89" x2="21.445" y2="12.7" width="0" layer="19" extent="1-1"/>
-<wire x1="10.13" y1="13.65" x2="21.445" y2="12.7" width="0" layer="19" extent="1-1"/>
-<wire x1="10.13" y1="11.75" x2="10.13" y2="13.65" width="0" layer="19" extent="1-1"/>
-<wire x1="9.93" y1="5.08" x2="10.13" y2="11.75" width="0" layer="19" extent="1-1"/>
-<wire x1="6.985" y1="29.355" x2="10.13" y2="13.65" width="0" layer="19" extent="1-1"/>
+<wire x1="13.015" y1="12.73" x2="21.445" y2="12.7" width="0" layer="19" extent="1-1"/>
+<wire x1="11.115" y1="12.73" x2="13.015" y2="12.73" width="0" layer="19" extent="1-1"/>
+<wire x1="8.485" y1="12.7" x2="11.115" y2="12.73" width="0" layer="19" extent="1-1"/>
+<wire x1="6.985" y1="25.255" x2="13.015" y2="12.73" width="0" layer="19" extent="1-1"/>
 </signal>
 <signal name="LOGIC_V+">
@@
 <contactref element="U$2" pad="VIN"/>
 <contactref element="D9" pad="A"/>
-<wire x1="12.73" y1="13.65" x2="8.89" y2="39.86" width="0" layer="19" extent="1-1"/>
-<wire x1="6.58" y1="12.7" x2="12.73" y2="13.65" width="0" layer="19" extent="1-1"/>
-<wire x1="17.78" y1="2.54" x2="12.73" y2="13.65" width="0" layer="19" extent="1-1"/>
+<wire x1="13.015" y1="10.13" x2="8.89" y2="39.86" width="0" layer="19" extent="1-1"/>
+<wire x1="8.485" y1="6.35" x2="13.015" y2="10.13" width="0" layer="19" extent="1-1"/>
+<wire x1="17.78" y1="2.54" x2="13.015" y2="10.13" width="0" layer="19" extent="1-1"/>
 </signal>
 <signal name="XCOND_EN">
@@
 <contactref element="D1" pad="C"/>
 <contactref element="D2" pad="A"/>
-<wire x1="6.985" y1="25.255" x2="9.93" y2="29.21" width="0" layer="19" extent="1-1"/>
-<wire x1="3.175" y1="29.355" x2="6.985" y2="25.255" width="0" layer="19" extent="1-1"/>
+<wire x1="3.175" y1="29.355" x2="6.985" y2="29.355" width="0.4064" layer="1"/>
+<wire x1="6.985" y1="29.355" x2="9.93" y2="29.355" width="0.4064" layer="1"/>
+<wire x1="9.93" y1="29.355" x2="9.93" y2="29.21" width="0.4064" layer="1"/>
 </signal>
 <signal name="N$5">
@@
 <contactref element="D3" pad="A"/>
 <wire x1="3.175" y1="25.255" x2="9.93" y2="24.13" width="0" layer="19" extent="1-1"/>
-<wire x1="3.175" y1="21.1" x2="3.175" y2="25.255" width="0" layer="19" extent="1-1"/>
+<wire x1="3.175" y1="21.1" x2="3.175" y2="25.255" width="0.4064" layer="1"/>
 </signal>
 <signal name="PUMP_PWM#">
@@
 <contactref element="D3" pad="C"/>
 <wire x1="36.83" y1="10.48" x2="44.45" y2="10.48" width="0" layer="19" extent="1-1"/>
-<wire x1="9.93" y1="17.145" x2="36.83" y2="10.48" width="0" layer="19" extent="1-1"/>
-<wire x1="3.175" y1="17" x2="9.93" y2="17.145" width="0" layer="19" extent="1-1"/>
+<wire x1="6.985" y1="16.915" x2="36.83" y2="10.48" width="0" layer="19" extent="1-1"/>
+<wire x1="3.175" y1="17" x2="7.62" y2="17" width="0.4064" layer="1"/>
+<wire x1="7.62" y1="17" x2="7.62" y2="17.145" width="0.4064" layer="1"/>
+<wire x1="7.62" y1="17.145" x2="6.985" y2="16.915" width="0" layer="19" extent="1-16"/>
 </signal>
 <signal name="N$1">
@@
 <contactref element="SPI_CON" pad="6"/>
 <contactref element="D9" pad="C"/>
-<wire x1="8.89" y1="43.96" x2="8.89" y2="46.99" width="0" layer="19" extent="1-1"/>
+<wire x1="8.89" y1="43.96" x2="8.89" y2="46.99" width="0.4064" layer="1"/>
 </signal>
 <signal name="SPI_CS">
@@
 <contactref element="R7" pad="2"/>
 <contactref element="R8" pad="1"/>
-<wire x1="29.21" y1="32.7" x2="33.02" y2="35.56" width="0" layer="19" extent="1-1"/>
-<wire x1="33.02" y1="27.94" x2="29.21" y2="32.7" width="0" layer="19" extent="1-1"/>
-<wire x1="29.21" y1="25.72" x2="33.02" y2="27.94" width="0" layer="19" extent="1-1"/>
-<wire x1="33.02" y1="15.24" x2="29.21" y2="25.72" width="0" layer="19" extent="1-1"/>
+<wire x1="33.02" y1="15.24" x2="29.21" y2="15.24" width="0.4064" layer="1"/>
+<wire x1="29.21" y1="15.24" x2="29.21" y2="25.72" width="0.4064" layer="1"/>
+<wire x1="33.02" y1="27.94" x2="31.115" y2="27.94" width="0.4064" layer="1"/>
+<wire x1="31.115" y1="27.94" x2="31.115" y2="32.385" width="0.4064" layer="1"/>
+<wire x1="31.115" y1="32.385" x2="29.21" y2="32.385" width="0.4064" layer="1"/>
+<wire x1="29.21" y1="32.385" x2="29.21" y2="32.7" width="0.4064" layer="1"/>
+<wire x1="29.21" y1="25.72" x2="31.115" y2="27.94" width="0" layer="19" extent="1-1"/>
+<wire x1="33.02" y1="35.56" x2="31.75" y2="35.56" width="0.4064" layer="1"/>
+<wire x1="31.75" y1="35.56" x2="31.75" y2="34.29" width="0.4064" layer="1"/>
+<wire x1="31.75" y1="34.29" x2="31.115" y2="34.29" width="0.4064" layer="1"/>
+<wire x1="31.115" y1="34.29" x2="31.115" y2="32.385" width="0.4064" layer="1"/>
 </signal>
 <signal name="SPI_SCK">
@@
 <contactref element="U$2" pad="23/A9"/>
 <contactref element="U$2" pad="3"/>
-<wire x1="29.21" y1="30.8" x2="33.02" y2="33.02" width="0" layer="19" extent="16-16"/>
-<wire x1="29.21" y1="27.62" x2="29.21" y2="30.8" width="0" layer="19" extent="16-16"/>
-<wire x1="33.02" y1="12.7" x2="29.21" y2="27.62" width="0" layer="19" extent="16-16"/>
-<wire x1="17.78" y1="10.16" x2="33.02" y2="12.7" width="0" layer="19" extent="1-1"/>
+<wire x1="33.02" y1="33.02" x2="31.115" y2="33.02" width="0.4064" layer="16"/>
+<wire x1="31.115" y1="33.02" x2="31.115" y2="30.48" width="0.4064" layer="16"/>
+<wire x1="31.115" y1="30.48" x2="29.21" y2="30.48" width="0.4064" layer="16"/>
+<wire x1="29.21" y1="30.48" x2="29.21" y2="30.8" width="0.4064" layer="16"/>
+<wire x1="29.21" y1="30.8" x2="29.21" y2="27.62" width="0.4064" layer="16"/>
+<wire x1="33.02" y1="12.7" x2="31.115" y2="12.7" width="0.4064" layer="16"/>
+<wire x1="31.115" y1="12.7" x2="31.115" y2="30.48" width="0.4064" layer="16"/>
+<wire x1="17.78" y1="10.16" x2="31.115" y2="12.7" width="0" layer="19" extent="16-16"/>
 </signal>
 <signal name="N$8">
 <contactref element="IC1" pad="4"/>
 <contactref element="C2" pad="1"/>
-<wire x1="12.43" y1="8.89" x2="12.73" y2="11.75" width="0" layer="19" extent="1-1"/>
+<wire x1="7.985" y1="9.525" x2="11.115" y2="10.13" width="0" layer="19" extent="1-1"/>
 </signal>
 <signal name="MCU_ADC0">

Commit message: update routing
Parts:
- moved D9 36.8 mm to (8.89, 5.08), flipped to the bottom
- moved LOAD_CON 15.5 mm to (39.4, 47.0), turned to 180 degrees
- moved D5 14.7 mm to (8.89, 10.2), turned to 90 degrees
- moved D8 9.86 mm to (14.0, 10.2), turned to 90 degrees
- moved IC1 7.85 mm to (10.2, 3.81)
- moved C3 7.43 mm to (14.0, 3.81), turned to 90 degrees
- moved C2 5.71 mm to (6.99, 3.81), turned to 90 degrees
- moved POW1_CON 5.08 mm to (33.0, 47.0)
- moved C1 4.96 mm to (3.81, 8.89)
- moved R6 2.54 mm to (29.2, 24.1)
- moved R7 2.54 mm to (29.2, 24.1)
- moved C4 2.54 mm to (11.4, 31.8)
- moved C5 2.54 mm to (11.4, 21.6)
- moved D1 1.27 mm to (6.99, 28.6)
- moved D2 1.27 mm to (3.17, 28.6)
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Connections:
- net SPI_CS: now also SPI_CON.4; no longer SPI_CON.2
- net SPI_MISO: now also SPI_CON.2; no longer SPI_CON.3
- net SPI_MOSI: now also SPI_CON.3; no longer SPI_CON.4
Routing:
- net POW1_V+: track 6.41 -> 86.0 mm, vias 0 -> 1
- net POW0_V+: track 6.41 -> 77.6 mm, vias 0 -> 1
- net MCU_V+: track 0.00 -> 69.4 mm, vias 0 -> 3
- net PUMP_V+: track 4.59 -> 44.5 mm, vias 0 -> 1
- net SPI_V+: track 3.03 -> 39.9 mm
- net POW01_V+: track 0.00 -> 30.4 mm, vias 0 -> 2
- net SPI_SCK: track 0.00 -> 20.3 mm
- net POW0_VMON: track 29.5 -> 46.4 mm
- net LOGIC_V+: track 0.00 -> 16.3 mm
- net LOAD_V+: track 27.9 -> 43.2 mm
- net GND: track 0.00 -> 8.13 mm
- net N$5: track 4.15 -> 12.2 mm
- net POW1_EN: track 11.7 -> 17.2 mm
- net N$1: track 35.6 -> 30.3 mm
- net N$2: track 35.6 -> 30.3 mm
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