File: eagle/main.brd (EAGLE design)
At the start: 49.2 x 49.5 mm, 34 parts, among them IC1 TS5205, Q1 SI4840DY, Q5 SI4840DY, U1 SN74AHC1G00DCKR, U2 SN74AHC1G00DCKR, U3 SN74AHC1G00DCKR

Commit message: update routing
Parts:
- moved D3 5.75 mm to (8.89, 19.7)
- moved D2 5.72 mm to (8.89, 28.6)
- moved C6 2.62 mm to (4.45, 19.1)
- moved D1 2.54 mm to (4.45, 28.6)
- moved C4 1.91 mm to (13.3, 31.8)
- moved C5 1.91 mm to (13.3, 21.6)
- turned C8 to 270 degrees
Routing:
- net GND: track 8.13 -> 0.00 mm
- net POW01_V+: track 30.4 -> 36.9 mm, vias 2 -> 0
- net LOAD_V+: track 43.2 -> 38.1 mm
- net N$4: track 7.18 -> 12.0 mm
- net N$5: track 12.2 -> 8.68 mm
- net PUMP_PWM#: track 8.66 -> 6.75 mm
- net PUMP_PWM: track 8.66 -> 6.75 mm
- net PUMP_V+: track 44.5 -> 43.8 mm
Changed lines of the file:
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@@
 <element name="T3" library="transistor" package="SOT23-BEC" value="" x="45.72" y="17.145" rot="MR0"/>
 <element name="T4" library="transistor" package="SOT23-BEC" value="" x="38.1" y="17.145" rot="MR0"/>
-<element name="C8" library="Panasonic-EEEFK_EEEFP" package="CAPAE660X800N" value="100UF" x="41.91" y="24.13">
-<attribute name="PACKAGE" value="CASE-D8" x="41.91" y="24.13" size="1.778" layer="27" display="off"/>
-<attribute name="OC_NEWARK" value="23T0852" x="41.91" y="24.13" size="1.778" layer="27" display="off"/>
-<attribute name="TOLERANCE" value="±20 %" x="41.91" y="24.13" size="1.778" layer="27" display="off"/>
-<attribute name="MPN" value="EEE-FK1E101XP" x="41.91" y="24.13" size="1.778" layer="27" display="off"/>
-<attribute name="SUPPLIER" value="PANASONIC" x="41.91" y="24.13" size="1.778" layer="27" display="off"/>
-<attribute name="VOLTAGERATING" value="25V" x="41.91" y="24.13" size="1.778" layer="27" display="off"/>
-<attribute name="OC_FARNELL" value="1850109  " x="41.91" y="24.13" size="1.778" layer="27" display="off"/>
+<element name="C8" library="Panasonic-EEEFK_EEEFP" package="CAPAE660X800N" value="100UF" x="41.91" y="24.13" rot="R270">
+<attribute name="PACKAGE" value="CASE-D8" x="41.91" y="24.13" size="1.778" layer="27" rot="R270" display="off"/>
+<attribute name="OC_NEWARK" value="23T0852" x="41.91" y="24.13" size="1.778" layer="27" rot="R270" display="off"/>
+<attribute name="TOLERANCE" value="±20 %" x="41.91" y="24.13" size="1.778" layer="27" rot="R270" display="off"/>
+<attribute name="MPN" value="EEE-FK1E101XP" x="41.91" y="24.13" size="1.778" layer="27" rot="R270" display="off"/>
+<attribute name="SUPPLIER" value="PANASONIC" x="41.91" y="24.13" size="1.778" layer="27" rot="R270" display="off"/>
+<attribute name="VOLTAGERATING" value="25V" x="41.91" y="24.13" size="1.778" layer="27" rot="R270" display="off"/>
+<attribute name="OC_FARNELL" value="1850109  " x="41.91" y="24.13" size="1.778" layer="27" rot="R270" display="off"/>
 </element>
 <element name="D5" library="diode" package="DO214AC" value="" x="8.89" y="10.16" rot="R90"/>
 <element name="D8" library="diode" package="DO214AC" value="" x="13.97" y="10.16" rot="R90"/>
 <element name="D9" library="diode" package="DO214AC" value="" x="8.89" y="5.08" rot="MR270"/>
-<element name="C4" library="rcl" package="C1210K" value="4.7u" x="11.43" y="31.75"/>
-<element name="C5" library="rcl" package="C1210K" value="4.7u" x="11.43" y="21.59"/>
-<element name="C6" library="rcl" package="C1210K" value="4.7u" x="6.985" y="18.415" rot="R90"/>
-<element name="D1" library="diode" package="DO214AC" value="" x="6.985" y="28.575" rot="R270"/>
-<element name="D2" library="diode" package="DO214AC" value="" x="3.175" y="28.575" rot="R90"/>
-<element name="D3" library="diode" package="DO214AC" value="" x="3.175" y="19.05" rot="R90"/>
+<element name="C4" library="rcl" package="C1210K" value="4.7u" x="13.335" y="31.75"/>
+<element name="C5" library="rcl" package="C1210K" value="4.7u" x="13.335" y="21.59"/>
+<element name="C6" library="rcl" package="C1210K" value="4.7u" x="4.445" y="19.05" rot="R90"/>
+<element name="D1" library="diode" package="DO214AC" value="" x="4.445" y="28.575" rot="R270"/>
+<element name="D2" library="diode" package="DO214AC" value="" x="8.89" y="28.575" rot="R90"/>
+<element name="D3" library="diode" package="DO214AC" value="" x="8.89" y="19.685" rot="R90"/>
 </elements>
 <signals>
@@
 <contactref element="C6" pad="2"/>
 <polygon width="0.4064" layer="1" isolate="0.4064">
-<vertex x="-0.635" y="50.165"/>
+<vertex x="-0.635" y="49.53"/>
 <vertex x="49.53" y="49.53"/>
 <vertex x="49.53" y="0"/>
@@
 </polygon>
 <polygon width="0.4064" layer="16">
-<vertex x="-0.635" y="50.165"/>
+<vertex x="0" y="50.165"/>
 <vertex x="49.53" y="49.53"/>
 <vertex x="49.53" y="0"/>
 <vertex x="0" y="0"/>
 </polygon>
-<wire x1="44.323" y1="24.13" x2="42.545" y2="24.13" width="0.4064" layer="1"/>
-<wire x1="42.545" y1="24.13" x2="42.545" y2="30.48" width="0.4064" layer="1"/>
 <wire x1="41.2496" y1="6.5786" x2="44.6786" y2="8.2804" width="0" layer="19" extent="16-16"/>
 <wire x1="37.0586" y1="8.2804" x2="41.2496" y2="6.5786" width="0" layer="19" extent="16-16"/>
+<wire x1="41.91" y1="21.717" x2="44.77" y2="16.045" width="0" layer="19" extent="1-16"/>
 <wire x1="29.21" y1="29.53" x2="25.4" y2="35.56" width="0" layer="19" extent="1-1"/>
 <wire x1="29.21" y1="23.18" x2="29.21" y2="29.53" width="0" layer="19" extent="1-16"/>
-<wire x1="44.323" y1="24.13" x2="44.77" y2="16.045" width="0" layer="19" extent="1-16"/>
 </signal>
 <signal name="POW01_V+">
@@
 <wire x1="8.89" y1="8.89" x2="8.89" y2="8.11" width="0.4064" layer="1"/>
 <wire x1="13.97" y1="8.11" x2="8.89" y2="8.11" width="0.4064" layer="1"/>
-<wire x1="6.985" y1="26.525" x2="6.985" y2="24.13" width="0.4064" layer="1"/>
-<via x="6.985" y="24.13" extent="1-16" drill="0.6" shape="square"/>
-<wire x1="6.985" y1="24.13" x2="6.985" y2="13.97" width="0.4064" layer="16"/>
-<via x="6.985" y="13.97" extent="1-16" drill="0.6" shape="square"/>
-<wire x1="6.985" y1="13.97" x2="6.985" y2="8.89" width="0.4064" layer="1"/>
+<wire x1="4.445" y1="26.525" x2="2.54" y2="26.67" width="0.4064" layer="1"/>
+<wire x1="6.985" y1="12.065" x2="6.985" y2="8.89" width="0.4064" layer="1"/>
 <wire x1="8.89" y1="8.11" x2="9.21" y2="8.11" width="0.4064" layer="1"/>
 <wire x1="9.21" y1="8.11" x2="9.21" y2="5.11" width="0.4064" layer="1"/>
+<wire x1="6.985" y1="12.065" x2="2.54" y2="12.065" width="0.4064" layer="1"/>
+<wire x1="2.54" y1="12.065" x2="2.54" y2="26.67" width="0.4064" layer="1"/>
 <wire x1="9.21" y1="5.11" x2="11.11" y2="5.11" width="0" layer="19" extent="1-1"/>
 </signal>
@@
 <wire x1="37.465" y1="36.77" x2="36.83" y2="36.77" width="0.4064" layer="1"/>
 <wire x1="45.085" y1="33.02" x2="45.085" y2="36.77" width="0.4064" layer="1"/>
-<wire x1="39.497" y1="24.13" x2="36.83" y2="24.13" width="0.4064" layer="1"/>
-<wire x1="36.83" y1="24.13" x2="36.83" y2="33.02" width="0.4064" layer="1"/>
+<wire x1="41.91" y1="26.543" x2="41.91" y2="33.02" width="0.4064" layer="1"/>
 <wire x1="36.83" y1="33.02" x2="36.83" y2="36.77" width="0.4064" layer="1"/>
 <wire x1="40.64" y1="46.99" x2="41.91" y2="46.99" width="0.4064" layer="1"/>
@@
 <contactref element="D1" pad="C"/>
 <contactref element="D2" pad="A"/>
-<wire x1="3.175" y1="30.625" x2="6.985" y2="30.625" width="0.4064" layer="1"/>
-<wire x1="6.985" y1="30.625" x2="8.66" y2="30.625" width="0.4064" layer="1"/>
-<wire x1="8.66" y1="30.625" x2="9.93" y2="31.75" width="0.4064" layer="1"/>
+<wire x1="8.89" y1="30.625" x2="4.445" y2="30.625" width="0.4064" layer="1"/>
+<wire x1="4.445" y1="30.625" x2="8.66" y2="30.625" width="0.4064" layer="1"/>
+<wire x1="8.66" y1="30.625" x2="11.835" y2="31.75" width="0.4064" layer="1"/>
 </signal>
 <signal name="N$5">
@@
 <contactref element="D2" pad="C"/>
 <contactref element="D3" pad="A"/>
-<wire x1="3.175" y1="21.1" x2="3.175" y2="21.59" width="0.4064" layer="1"/>
-<wire x1="3.175" y1="21.59" x2="3.175" y2="26.525" width="0.4064" layer="1"/>
-<wire x1="9.93" y1="21.59" x2="3.175" y2="21.59" width="0.4064" layer="1"/>
+<wire x1="8.89" y1="21.735" x2="8.89" y2="24.13" width="0.4064" layer="1"/>
+<wire x1="8.89" y1="24.13" x2="8.89" y2="26.525" width="0.4064" layer="1"/>
+<wire x1="11.835" y1="21.59" x2="8.89" y2="24.13" width="0.4064" layer="1"/>
 </signal>
 <signal name="PUMP_PWM#">
 <contactref element="U$2" pad="17/A3"/>
 <contactref element="C5" pad="2"/>
-<wire x1="17.78" y1="25.4" x2="12.93" y2="25.4" width="0.4064" layer="1"/>
-<wire x1="12.93" y1="25.4" x2="12.93" y2="21.59" width="0.4064" layer="1"/>
+<wire x1="17.78" y1="25.4" x2="14.835" y2="25.4" width="0.4064" layer="1"/>
+<wire x1="14.835" y1="25.4" x2="14.835" y2="21.59" width="0.4064" layer="1"/>
 </signal>
 <signal name="PUMP_V+">
@@
 <contactref element="C6" pad="1"/>
 <contactref element="D3" pad="C"/>
-<wire x1="3.175" y1="17" x2="7.62" y2="17" width="0.4064" layer="1"/>
+<wire x1="8.89" y1="17.635" x2="7.62" y2="17" width="0.4064" layer="1"/>
 <wire x1="7.62" y1="17" x2="7.62" y2="17.145" width="0.4064" layer="1"/>
 <wire x1="36.83" y1="10.48" x2="34.29" y2="10.48" width="0.4064" layer="16"/>
@@
 <via x="10.795" y="17.145" extent="1-16" drill="0.6" shape="square"/>
 <wire x1="10.795" y1="17.145" x2="6.985" y2="17.145" width="0.4064" layer="1"/>
-<wire x1="6.985" y1="17.145" x2="6.985" y2="16.915" width="0.4064" layer="1"/>
+<wire x1="6.985" y1="17.145" x2="4.445" y2="17.55" width="0.4064" layer="1"/>
 <wire x1="36.83" y1="10.48" x2="44.45" y2="10.48" width="0" layer="19" extent="16-16"/>
 <wire x1="7.62" y1="17.145" x2="6.985" y2="17.145" width="0" layer="19" extent="1-1"/>
@@
 <contactref element="U$2" pad="16/A2"/>
 <contactref element="C4" pad="2"/>
-<wire x1="17.78" y1="27.94" x2="12.93" y2="27.94" width="0.4064" layer="1"/>
-<wire x1="12.93" y1="27.94" x2="12.93" y2="31.75" width="0.4064" layer="1"/>
+<wire x1="17.78" y1="27.94" x2="14.835" y2="27.94" width="0.4064" layer="1"/>
+<wire x1="14.835" y1="27.94" x2="14.835" y2="31.75" width="0.4064" layer="1"/>
 </signal>
 <signal name="POW0_VMON">
@@
 <wire x1="41.91" y1="4.445" x2="41.91" y2="6.5786" width="0.4064" layer="16"/>
 </signal>
-<signal name="N$9">
-<via x="42.545" y="30.48" extent="1-16" drill="0.6" shape="square"/>
-</signal>
 </signals>

Commit message: routing
Parts:
- removed SPI_CON: (no value), pinhead:1X06
- moved D8 34.6 mm to (26.0, 42.5), turned to 0 degrees
- moved D5 33.9 mm to (26.0, 39.4), turned to 0 degrees
- moved C6 8.91 mm to (13.3, 19.7), flipped to the bottom, turned to 180 degrees
- moved R7 8.64 mm to (36.2, 29.2), flipped to the bottom
- moved R8 7.96 mm to (36.2, 34.3)
- moved R2 7.85 mm to (39.4, 13.3), flipped to the top
- moved POW0_CON 7.10 mm to (38.7, 45.7)
- moved LOAD_CON 5.85 mm to (45.1, 45.7)
- moved R1 5.43 mm to (44.5, 13.3)
- moved C8 5.08 mm to (41.9, 29.2)
- moved T3 4.26 mm to (41.9, 19.1), flipped to the top
- moved U2 4.26 mm to (41.9, 9.53), flipped to the top
- moved T4 4.26 mm to (41.9, 19.1)
- moved U3 4.26 mm to (41.9, 9.53)
- moved Q5 3.81 mm to (41.9, 39.4)
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Connections:
- net GND: no longer SPI_CON.1
- net SPI_CS: no longer SPI_CON.4
- net SPI_MISO: no longer SPI_CON.2
- net SPI_MOSI: no longer SPI_CON.3
- net SPI_SCK: no longer SPI_CON.5
- net SPI_V+: no longer SPI_CON.6
Routing:
- net POW1_V+: track 86.0 -> 32.6 mm, vias 1 -> 0
- net POW0_V+: track 77.6 -> 31.3 mm
- net SPI_V+: track 39.9 -> 0.00 mm
- net POW01_V+: track 36.9 -> 76.1 mm
- net SPI_SCK: track 20.3 -> 0.00 mm
- net PUMP_V+: track 43.8 -> 56.4 mm, vias 1 -> 2
- net LOAD_V+: track 38.1 -> 31.9 mm
- net GND: track 0.00 -> 4.78 mm, vias 0 -> 1
- net N$2: track 30.3 -> 25.8 mm, vias 1 -> 0
- net N$1: track 30.3 -> 25.8 mm, vias 1 -> 0
- net LOGIC_V+: track 16.3 -> 20.1 mm
- net MCU_V+: track 69.4 -> 65.7 mm, vias 3 -> 1
- net XCOND_EN: track 8.66 -> 10.8 mm, vias 0 -> 1
- net PUMP_PWM#: track 6.75 -> 4.85 mm
- net PUMP_PWM: track 6.75 -> 4.85 mm
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
Commit message: routing
Parts:
- moved IC1 6.25 mm to (7.62, 10.8)
- moved D9 3.24 mm to (12.1, 4.45)
- moved C1 2.54 mm to (3.81, 12.7)
- moved C3 2.29 mm to (12.1, 5.08)
- moved C4 2.01 mm to (11.4, 29.2)
- moved C5 1.91 mm to (11.4, 23.5)
- moved C6 1.91 mm to (11.4, 19.7)
- moved C2 1.91 mm to (7.62, 5.08), turned to 270 degrees
- moved D3 1.27 mm to (6.99, 19.7)
- moved R5 1.27 mm to (27.9, 30.5)
- moved R6 1.27 mm to (27.9, 24.1)
- moved U$2 1.27 mm to (24.1, 19.1)
Routing:
- net POW01_V+: track 76.1 -> 64.6 mm
- net PUMP_V+: track 56.4 -> 51.7 mm
- net N$4: track 10.2 -> 6.26 mm
- net MCU_V+: track 65.7 -> 62.5 mm
- net POW1_EN: track 18.3 -> 20.9 mm
- net POW0_VMON: track 46.4 -> 44.0 mm
- net POW0_EN: track 16.5 -> 17.8 mm
- net N$5: track 7.51 -> 6.46 mm
- net N$8: track 3.56 -> 4.36 mm
- net POW1_VMON: track 33.3 -> 34.1 mm
- net LOGIC_V+: track 20.1 -> 19.4 mm
- net PUMP_PWM#: track 4.85 -> 5.48 mm
- net POW0_V+: track 31.3 -> 31.8 mm

Commit message: routing
Routing:
- net POW01_V+: track 64.6 -> 62.0 mm
Changed lines of the file:
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@@
 <wire x1="23.985" y1="42.545" x2="23.985" y2="39.37" width="0.4064" layer="1"/>
 <wire x1="23.985" y1="39.37" x2="24.13" y2="39.37" width="0.4064" layer="1"/>
-<wire x1="22.225" y1="13.97" x2="8.89" y2="13.97" width="0.4064" layer="1"/>
+<wire x1="22.225" y1="18.415" x2="17.78" y2="13.97" width="0.4064" layer="1"/>
+<wire x1="17.78" y1="13.97" x2="8.89" y2="13.97" width="0.4064" layer="1"/>
 <wire x1="8.89" y1="13.97" x2="6.35" y2="13.97" width="0.4064" layer="1"/>
 <wire x1="8.57" y1="12.095" x2="8.89" y2="12.095" width="0.4064" layer="1"/>
@@
 <wire x1="6.35" y1="13.97" x2="3.81" y2="13.97" width="0.4064" layer="1"/>
 <wire x1="3.81" y1="13.97" x2="3.81" y2="14.2" width="0.4064" layer="1"/>
-<wire x1="22.225" y1="13.97" x2="22.225" y2="39.37" width="0.4064" layer="1"/>
+<wire x1="22.225" y1="18.415" x2="22.225" y2="39.37" width="0.4064" layer="1"/>
 <wire x1="22.225" y1="39.37" x2="23.985" y2="39.37" width="0.4064" layer="1"/>
 </signal>

Commit message: power terminals
Parts:
- moved LOAD_CON 1.27 mm to (43.8, 45.7)
- moved POW1_CON 1.27 mm to (33.7, 45.7)
Routing:
- net LOAD_V+: track 31.9 -> 29.4 mm
Changed lines of the file:
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@@
 <elements>
 <element name="POW0_CON" library="pinhead" package="1X02" value="" x="38.735" y="45.72" rot="R180"/>
-<element name="POW1_CON" library="pinhead" package="1X02" value="" x="32.385" y="45.72" rot="R180"/>
-<element name="LOAD_CON" library="pinhead" package="1X02" value="" x="45.085" y="45.72" rot="R180"/>
+<element name="POW1_CON" library="pinhead" package="1X02" value="" x="33.655" y="45.72" rot="R180"/>
+<element name="LOAD_CON" library="pinhead" package="1X02" value="" x="43.815" y="45.72" rot="R180"/>
 <element name="C1" library="rcl" package="C1210K" value="4.7u" x="3.81" y="12.7" rot="R270"/>
 <element name="R2" library="resistor" package="M0805" value="100K" x="39.37" y="13.335" rot="R90"/>
@@
 <contactref element="C6" pad="2"/>
 <polygon width="0.4064" layer="1" isolate="0.4064">
-<vertex x="0" y="50.165"/>
+<vertex x="0" y="50.8"/>
 <vertex x="49.53" y="49.53"/>
 <vertex x="49.53" y="0"/>
@@
 </polygon>
 <polygon width="0.4064" layer="16">
-<vertex x="0" y="50.165"/>
+<vertex x="0" y="50.8"/>
 <vertex x="49.53" y="49.53"/>
 <vertex x="49.53" y="0"/>
@@
 <contactref element="R7" pad="1"/>
 <contactref element="D8" pad="A"/>
-<wire x1="33.655" y1="45.72" x2="33.655" y2="42.545" width="0.4064" layer="1"/>
-<wire x1="33.655" y1="45.72" x2="33.655" y2="41.91" width="0.4064" layer="16"/>
-<wire x1="33.655" y1="41.91" x2="36.195" y2="41.91" width="0.4064" layer="16"/>
+<wire x1="34.925" y1="45.72" x2="34.925" y2="42.545" width="0.4064" layer="1"/>
+<wire x1="34.925" y1="45.72" x2="34.925" y2="41.91" width="0.4064" layer="16"/>
+<wire x1="34.925" y1="41.91" x2="36.195" y2="41.91" width="0.4064" layer="16"/>
 <wire x1="36.195" y1="41.91" x2="41.91" y2="41.91" width="0.4064" layer="16"/>
 <wire x1="41.91" y1="41.91" x2="41.91" y2="41.97" width="0.4064" layer="16"/>
-<wire x1="28.085" y1="42.545" x2="33.655" y2="42.545" width="0.4064" layer="1"/>
+<wire x1="28.085" y1="42.545" x2="34.925" y2="42.545" width="0.4064" layer="1"/>
 <wire x1="36.195" y1="30.16" x2="36.195" y2="41.91" width="0.4064" layer="16"/>
 </signal>
@@
 <contactref element="C8" pad="1"/>
 <wire x1="41.91" y1="31.623" x2="41.91" y2="36.77" width="0.4064" layer="1"/>
-<wire x1="46.355" y1="45.72" x2="46.355" y2="36.83" width="0.4064" layer="16"/>
-<wire x1="46.355" y1="36.83" x2="42.545" y2="36.83" width="0.4064" layer="16"/>
+<wire x1="45.085" y1="45.72" x2="45.085" y2="36.83" width="0.4064" layer="16"/>
+<wire x1="45.085" y1="36.83" x2="42.545" y2="36.83" width="0.4064" layer="16"/>
 <wire x1="42.545" y1="36.83" x2="42.545" y2="36.77" width="0.4064" layer="16"/>
-<wire x1="41.91" y1="36.83" x2="46.355" y2="36.83" width="0.4064" layer="1"/>
-<wire x1="46.355" y1="36.83" x2="46.355" y2="45.72" width="0.4064" layer="1"/>
+<wire x1="41.91" y1="36.83" x2="45.085" y2="36.83" width="0.4064" layer="1"/>
+<wire x1="45.085" y1="36.83" x2="45.085" y2="45.72" width="0.4064" layer="1"/>
 <wire x1="41.275" y1="36.77" x2="41.91" y2="36.77" width="0.4064" layer="1"/>
 <wire x1="41.91" y1="36.77" x2="41.91" y2="36.83" width="0.4064" layer="1"/>

Commit message: routing
Parts:
- moved Q1 2.54 mm to (41.9, 36.8)
- moved Q5 2.54 mm to (41.9, 36.8)
- moved C8 1.91 mm to (41.9, 27.3)
- moved D5 1.27 mm to (24.8, 39.4)
- moved D8 1.27 mm to (24.8, 42.5)
Routing:
- net LOAD_V+: track 29.4 -> 38.3 mm
- net N$2: track 25.8 -> 23.3 mm
- net N$1: track 25.8 -> 23.3 mm
- net POW0_V+: track 31.8 -> 29.7 mm
- net POW1_V+: track 32.6 -> 33.7 mm

Commit message: routing
Parts:
- moved D9 2.29 mm to (10.2, 5.71)
- moved POW1_CON 1.27 mm to (32.4, 45.7)
- moved LOAD_CON 1.27 mm to (42.5, 45.7)
- moved POW0_CON 1.27 mm to (37.5, 45.7)
Routing:
- net LOAD_V+: track 38.3 -> 35.7 mm
- net LOGIC_V+: track 19.4 -> 21.9 mm
- net POW0_V+: track 29.7 -> 30.5 mm
- net POW1_V+: track 33.7 -> 33.1 mm
Changed lines of the file:
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@@
 </autorouter>
 <elements>
-<element name="POW0_CON" library="pinhead" package="1X02" value="" x="38.735" y="45.72" rot="R180"/>
-<element name="POW1_CON" library="pinhead" package="1X02" value="" x="33.655" y="45.72" rot="R180"/>
-<element name="LOAD_CON" library="pinhead" package="1X02" value="" x="43.815" y="45.72" rot="R180"/>
+<element name="POW0_CON" library="pinhead" package="1X02" value="" x="37.465" y="45.72" rot="R180"/>
+<element name="POW1_CON" library="pinhead" package="1X02" value="" x="32.385" y="45.72" rot="R180"/>
+<element name="LOAD_CON" library="pinhead" package="1X02" value="" x="42.545" y="45.72" rot="R180"/>
 <element name="C1" library="rcl" package="C1210K" value="4.7u" x="3.81" y="12.7" rot="R270"/>
 <element name="R2" library="resistor" package="M0805" value="100K" x="39.37" y="13.335" rot="R90"/>
@@
 <element name="D5" library="diode" package="DO214AC" value="" x="24.765" y="39.37"/>
 <element name="D8" library="diode" package="DO214AC" value="" x="24.765" y="42.545"/>
-<element name="D9" library="diode" package="DO214AC" value="" x="12.065" y="4.445" rot="MR270"/>
+<element name="D9" library="diode" package="DO214AC" value="" x="10.16" y="5.715" rot="MR270"/>
 <element name="C4" library="rcl" package="C1210K" value="4.7u" x="11.43" y="29.21"/>
 <element name="C5" library="rcl" package="C1210K" value="4.7u" x="11.43" y="23.495"/>
@@
 <wire x1="31.115" y1="39.37" x2="40.005" y2="39.37" width="0.4064" layer="1"/>
 <wire x1="26.815" y1="39.37" x2="31.115" y2="39.37" width="0.4064" layer="1"/>
-<wire x1="40.005" y1="45.72" x2="40.005" y2="41.335" width="1.016" layer="1"/>
-<wire x1="40.005" y1="41.335" x2="41.91" y2="39.43" width="1.016" layer="1"/>
+<wire x1="38.735" y1="45.72" x2="38.735" y2="41.97" width="1.016" layer="1"/>
+<wire x1="38.735" y1="41.97" x2="41.91" y2="39.43" width="1.016" layer="1"/>
 <wire x1="40.005" y1="39.37" x2="41.91" y2="39.43" width="0" layer="19" extent="1-1"/>
 </signal>
@@
 <vertex x="0" y="0"/>
 </polygon>
-<polygon width="0.4064" layer="16">
+<polygon width="0.4064" layer="16" isolate="0.3048">
 <vertex x="0" y="49.53"/>
 <vertex x="49.53" y="49.53"/>
@@
 <wire x1="14.605" y1="2.54" x2="14.605" y2="6.35" width="0.4064" layer="1"/>
 <wire x1="14.605" y1="6.35" x2="12.065" y2="6.35" width="0.4064" layer="1"/>
-<wire x1="16.51" y1="2.395" x2="12.065" y2="2.395" width="0.4064" layer="16"/>
 <wire x1="12.065" y1="6.35" x2="12.065" y2="6.58" width="0.4064" layer="1"/>
 <wire x1="12.065" y1="6.58" x2="11.43" y2="6.58" width="0.4064" layer="1"/>
@@
 <wire x1="11.43" y1="9.525" x2="8.57" y2="9.525" width="0.4064" layer="1"/>
 <wire x1="8.57" y1="9.525" x2="8.57" y2="9.495" width="0.4064" layer="1"/>
+<wire x1="16.51" y1="2.395" x2="12.065" y2="2.395" width="0.4064" layer="16"/>
+<wire x1="12.065" y1="2.395" x2="10.16" y2="3.81" width="0.4064" layer="16"/>
+<wire x1="10.16" y1="3.81" x2="10.16" y2="3.665" width="0.4064" layer="16"/>
 <wire x1="16.51" y1="2.395" x2="16.51" y2="2.54" width="0" layer="19" extent="16-16"/>
 </signal>
@@
 <contactref element="R7" pad="1"/>
 <contactref element="D8" pad="A"/>
-<wire x1="34.925" y1="45.72" x2="34.925" y2="42.545" width="0.4064" layer="1"/>
-<wire x1="26.815" y1="42.545" x2="34.925" y2="42.545" width="0.4064" layer="1"/>
+<wire x1="33.655" y1="45.72" x2="33.655" y2="42.545" width="0.4064" layer="1"/>
+<wire x1="26.815" y1="42.545" x2="33.655" y2="42.545" width="0.4064" layer="1"/>
 <wire x1="36.195" y1="30.16" x2="36.195" y2="40.005" width="0.4064" layer="16"/>
-<wire x1="34.925" y1="45.72" x2="34.925" y2="41.275" width="1.016" layer="16"/>
-<wire x1="34.925" y1="41.275" x2="36.195" y2="40.005" width="1.016" layer="16"/>
+<wire x1="33.655" y1="45.72" x2="33.655" y2="41.91" width="1.016" layer="16"/>
+<wire x1="33.655" y1="41.91" x2="36.195" y2="40.005" width="1.016" layer="16"/>
 <wire x1="36.195" y1="40.005" x2="41.91" y2="40.005" width="1.016" layer="16"/>
 <wire x1="41.91" y1="40.005" x2="41.91" y2="39.43" width="1.016" layer="16"/>
@@
 <contactref element="Q1" pad="1-3"/>
 <contactref element="C8" pad="1"/>
-<wire x1="41.91" y1="29.718" x2="41.91" y2="34.29" width="1.016" layer="1"/>
+<wire x1="41.91" y1="29.718" x2="41.91" y2="36.77" width="1.016" layer="1"/>
 <wire x1="41.91" y1="36.77" x2="41.91" y2="36.83" width="0.4064" layer="1"/>
-<wire x1="45.085" y1="45.72" x2="46.355" y2="45.72" width="1.016" layer="1"/>
-<wire x1="46.355" y1="45.72" x2="46.355" y2="36.83" width="1.016" layer="1"/>
-<wire x1="46.355" y1="36.83" x2="41.91" y2="36.83" width="1.016" layer="1"/>
-<wire x1="42.545" y1="34.23" x2="46.355" y2="34.23" width="1.016" layer="16"/>
-<wire x1="46.355" y1="34.23" x2="46.355" y2="45.72" width="1.016" layer="16"/>
-<wire x1="46.355" y1="45.72" x2="45.085" y2="45.72" width="1.016" layer="16"/>
-<wire x1="41.91" y1="36.77" x2="41.91" y2="34.29" width="1.016" layer="1"/>
-<wire x1="41.91" y1="34.29" x2="41.275" y2="34.23" width="0" layer="19" extent="1-1"/>
+<wire x1="43.815" y1="45.72" x2="45.72" y2="43.18" width="1.016" layer="1"/>
+<wire x1="45.72" y1="43.18" x2="45.72" y2="36.83" width="1.016" layer="1"/>
+<wire x1="45.72" y1="36.83" x2="41.91" y2="36.83" width="1.016" layer="1"/>
+<wire x1="42.545" y1="34.23" x2="45.72" y2="34.23" width="1.016" layer="16"/>
+<wire x1="45.72" y1="34.23" x2="45.72" y2="43.18" width="1.016" layer="16"/>
+<wire x1="45.72" y1="43.18" x2="43.815" y2="45.72" width="1.016" layer="16"/>
+<wire x1="42.545" y1="34.23" x2="41.275" y2="34.23" width="0" layer="19" extent="1-16"/>
 </signal>
 <signal name="N$4">
