File: eagle/main.brd (EAGLE design)
At the start: 49.2 x 49.5 mm, 33 parts, among them IC1 TS5205, Q1 SI4840DY, Q5 SI4840DY, U1 SN74AHC1G00DCKR, U2 SN74AHC1G00DCKR, U3 SN74AHC1G00DCKR

Commit message: silkscreen
Routing:
- net POW0_V+: track 30.5 -> 32.4 mm
- net LOAD_V+: track 35.7 -> 36.4 mm
Other:
- board text added: "+"
- board text added: "PSMUX 2094042fas349"
